File: Kicad/Eve/driver_stepper.kicad_sch (KiCad schematic)
At the start: 21 parts, among them J8 Conn_01x04, Q1 SQJ504EP-T1_GE3, Q6 SQJ504EP-T1_GE3, Q7 SQJ504EP-T1_GE3, Q8 SQJ504EP-T1_GE3, U3 TMC2590-TA

Commit message: empreinte 13/11
Parts:
- C23, C24, C29, C31: footprint (none) -> Capacitor_SMD:C_0603_1608Metric_Pad1.08x0.95mm_HandSolder
- Q1, Q6, Q7, Q8: footprint SQJ968EPT1GE3 -> Mosfet:SQJ968EPT1GE3
- R24, R9: footprint (none) -> Resistor_SMD:R_0603_1608Metric_Pad0.98x0.95mm_HandSolder
- R26, R27: value 0.075/2W -> 0.075; puissance (none) -> 2W
- U3: footprint TQFP32_7X7_TRI -> TMC2590:QFP50P700X700X114-33N
Other:
- moved on the sheet: R27
Changed lines of the file:
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@@
     (stroke (width 0) (type default))
   )
-  (wire (pts (xy 233.68 109.22) (xy 233.68 106.68))
+  (wire (pts (xy 233.68 109.22) (xy 233.68 105.41))
     (stroke (width 0) (type default))
   )
@@
     (stroke (width 0) (type default))
   )
-  (wire (pts (xy 233.68 95.25) (xy 233.68 99.06))
+  (wire (pts (xy 233.68 95.25) (xy 233.68 97.79))
     (stroke (width 0) (type default))
   )
@@
       (effects (font (size 1.27 1.27)))
     )
-    (property "Footprint" "SQJ968EPT1GE3" (at 205.74 29.54 0)
+    (property "Footprint" "Mosfet:SQJ968EPT1GE3" (at 205.74 29.54 0)
       (effects (font (size 1.27 1.27)) (justify left top) hide)
     )
@@
       (effects (font (size 1.27 1.27)))
     )
-    (property "Footprint" "SQJ968EPT1GE3" (at 266.7 214.3 0)
+    (property "Footprint" "Mosfet:SQJ968EPT1GE3" (at 266.7 214.3 0)
       (effects (font (size 1.27 1.27)) (justify left top) hide)
     )
@@
       (effects (font (size 1.27 1.27)) (justify left))
     )
-    (property "Footprint" "" (at 177.8 86.36 0)
+    (property "Footprint" "Capacitor_SMD:C_0603_1608Metric_Pad1.08x0.95mm_HandSolder" (at 177.8 86.36 0)
       (effects (font (size 1.27 1.27)) hide)
     )
@@
       (effects (font (size 1.524 1.524)))
     )
-    (property "Footprint" "TQFP32_7X7_TRI" (at 101.6 76.2 0)
+    (property "Footprint" "TMC2590:QFP50P700X700X114-33N" (at 101.6 76.2 0)
       (effects (font (size 1.27 1.27) italic) hide)
     )
@@
       (effects (font (size 1.27 1.27)) (justify left))
     )
-    (property "Footprint" "" (at 241.3 44.958 90)
+    (property "Footprint" "Resistor_SMD:R_0603_1608Metric_Pad0.98x0.95mm_HandSolder" (at 241.3 44.958 90)
       (effects (font (size 1.27 1.27)) hide)
     )
@@
       (effects (font (size 1.27 1.27)) (justify left))
     )
-    (property "Footprint" "" (at 35.56 52.07 0)
+    (property "Footprint" "Capacitor_SMD:C_0603_1608Metric_Pad1.08x0.95mm_HandSolder" (at 35.56 52.07 0)
       (effects (font (size 1.27 1.27)) hide)
     )
@@
       (effects (font (size 1.27 1.27)))
     )
-    (property "Footprint" "SQJ968EPT1GE3" (at 262.89 149.53 0)
+    (property "Footprint" "Mosfet:SQJ968EPT1GE3" (at 262.89 149.53 0)
       (effects (font (size 1.27 1.27)) (justify left top) hide)
     )
@@
       (effects (font (size 1.27 1.27)) (justify left))
     )
-    (property "Footprint" "" (at 132.08 48.26 0)
+    (property "Footprint" "Capacitor_SMD:C_0603_1608Metric_Pad1.08x0.95mm_HandSolder" (at 132.08 48.26 0)
       (effects (font (size 1.27 1.27)) hide)
     )
@@
       (effects (font (size 1.27 1.27)))
     )
-    (property "Footprint" "SQJ968EPT1GE3" (at 201.93 149.53 0)
+    (property "Footprint" "Mosfet:SQJ968EPT1GE3" (at 201.93 149.53 0)
       (effects (font (size 1.27 1.27)) (justify left top) hide)
     )
@@
       (effects (font (size 1.27 1.27)) (justify left))
     )
-    (property "Footprint" "" (at 49.53 52.07 0)
+    (property "Footprint" "Capacitor_SMD:C_0603_1608Metric_Pad1.08x0.95mm_HandSolder" (at 49.53 52.07 0)
       (effects (font (size 1.27 1.27)) hide)
     )
@@
     )
   )
-  (symbol (lib_id "Device:R") (at 233.68 102.87 180) (unit 1)
-    (in_bom yes) (on_board yes) (dnp no) (fields_autoplaced)
-    (property "Reference" "R27" (at 231.14 104.14 0)
-      (effects (font (size 1.27 1.27)) (justify left))
-    )
-    (property "Value" "0.075/2W" (at 231.14 101.6 0)
-      (effects (font (size 1.27 1.27)) (justify left))
-    )
-    (property "Footprint" "" (at 235.458 102.87 90)
-      (effects (font (size 1.27 1.27)) hide)
-    )
-    (property "Datasheet" "~" (at 233.68 102.87 0)
-      (effects (font (size 1.27 1.27)) hide)
+  (symbol (lib_id "Device:R") (at 233.68 101.6 180) (unit 1)
+    (in_bom yes) (on_board yes) (dnp no)
+    (property "Reference" "R27" (at 227.33 100.33 0)
+      (effects (font (size 1.27 1.27)) (justify right))
+    )
+    (property "Value" "0.075" (at 226.06 102.87 0)
+      (effects (font (size 1.27 1.27)) (justify right))
+    )
+    (property "Footprint" "" (at 235.458 101.6 90)
+      (effects (font (size 1.27 1.27)) hide)
+    )
+    (property "Datasheet" "~" (at 233.68 101.6 0)
+      (effects (font (size 1.27 1.27)) hide)
+    )
+    (property "puissance" "2W" (at 229.87 105.41 0)
+      (effects (font (size 1.27 1.27)))
     )
     (pin "1")
@@
   )
   (symbol (lib_id "Device:R") (at 233.68 36.83 180) (unit 1)
-    (in_bom yes) (on_board yes) (dnp no) (fields_autoplaced)
+    (in_bom yes) (on_board yes) (dnp no)
     (property "Reference" "R26" (at 231.14 38.1 0)
       (effects (font (size 1.27 1.27)) (justify left))
     )
-    (property "Value" "0.075/2W" (at 231.14 35.56 0)
+    (property "Value" "0.075" (at 231.14 35.56 0)
       (effects (font (size 1.27 1.27)) (justify left))
     )
@@
     (property "Datasheet" "~" (at 233.68 36.83 0)
       (effects (font (size 1.27 1.27)) hide)
+    )
+    (property "puissance" "2W" (at 228.6 33.02 0)
+      (effects (font (size 1.27 1.27) italic))
     )
     (pin "1")
@@
       (effects (font (size 1.27 1.27)) (justify left))
     )
-    (property "Footprint" "" (at 241.3 110.998 90)
-      (effects (font (size 1.27 1.27)) hide)
-    )
+    (property "Footprint" "Resistor_SMD:R_0603_1608Metric_Pad0.98x0.95mm_HandSolder" (at 241.3 110.998 90)
+      (effects (font (size 1.27 1.27)) hide)
+    )

Commit message: pulled main and started routing
Parts:
- removed D8: SMBJ54A, symbol Device:D_Schottky
- C25, C26, C27, C28: footprint (none) -> Capacitor_SMD:CP_Elec_10x10.5; MFR (none) -> 865060657011; Voltage 80V -> 50V
- C30, C50: footprint (none) -> Capacitor_SMD:C_0603_1608Metric_Pad1.08x0.95mm_HandSolder
- J8: footprint (none) -> Connector_Molex:Molex_Mini-Fit_Jr_5566-04A2_2x02_P4.20mm_Vertical
- R26, R27: footprint (none) -> Resistor_SMD:R_2512_6332Metric_Pad1.40x3.35mm_HandSolder
Changed lines of the file:
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@@
   (junction (at 49.53 48.26) (diameter 0) (color 0 0 0 0)
   )
-  (junction (at 58.42 48.26) (diameter 0) (color 0 0 0 0)
-  )
   (junction (at 175.26 86.36) (diameter 0) (color 0 0 0 0)
   )
@@
   (junction (at 233.68 95.25) (diameter 0) (color 0 0 0 0)
   )
-  (junction (at 58.42 55.88) (diameter 0) (color 0 0 0 0)
-  )
   (junction (at 81.28 48.26) (diameter 0) (color 0 0 0 0)
   )
@@
     (stroke (width 0) (type default))
   )
-  (wire (pts (xy 58.42 48.26) (xy 69.85 48.26))
-    (stroke (width 0) (type default))
-  )
   (wire (pts (xy 81.28 55.88) (xy 91.44 55.88))
     (stroke (width 0) (type default))
@@
     (stroke (width 0) (type default))
   )
-  (wire (pts (xy 69.85 55.88) (xy 58.42 55.88))
-    (stroke (width 0) (type default))
-  )
   (wire (pts (xy 270.51 123.19) (xy 270.51 124.46))
     (stroke (width 0) (type default))
@@
     (stroke (width 0) (type default))
   )
-  (wire (pts (xy 49.53 48.26) (xy 58.42 48.26))
+  (wire (pts (xy 49.53 48.26) (xy 69.85 48.26))
     (stroke (width 0) (type default))
   )
@@
     (stroke (width 0) (type default))
   )
-  (wire (pts (xy 58.42 55.88) (xy 49.53 55.88))
+  (wire (pts (xy 49.53 55.88) (xy 69.85 55.88))
     (stroke (width 0) (type default))
   )
@@
       (effects (font (size 1.27 1.27)) (justify left))
     )
-    (property "Footprint" "" (at 92.4052 55.88 0)
+    (property "Footprint" "Capacitor_SMD:CP_Elec_10x10.5" (at 92.4052 55.88 0)
       (effects (font (size 1.27 1.27)) hide)
     )
@@
       (effects (font (size 1.27 1.27)) hide)
     )
-    (property "Voltage" "80V" (at 91.44 45.72 0)
+    (property "Voltage" "50V" (at 91.44 45.72 0)
       (effects (font (size 1.27 1.27)))
     )
     (property "R" "45 mOhm" (at 91.44 43.18 0)
       (effects (font (size 1.27 1.27)))
+    )
+    (property "MFR" "865060657011" (at 91.44 52.07 90)
+      (effects (font (size 1.27 1.27)) hide)
     )
     (pin "1")
@@
       (effects (font (size 1.27 1.27)) (justify left))
     )
-    (property "Footprint" "" (at 114.3 52.07 0)
+    (property "Footprint" "Capacitor_SMD:C_0603_1608Metric_Pad1.08x0.95mm_HandSolder" (at 114.3 52.07 0)
       (effects (font (size 1.27 1.27)) hide)
     )
@@
       (effects (font (size 1.27 1.27)) (justify left))
     )
-    (property "Footprint" "" (at 102.5652 55.88 0)
+    (property "Footprint" "Capacitor_SMD:CP_Elec_10x10.5" (at 102.5652 55.88 0)
       (effects (font (size 1.27 1.27)) hide)
     )
@@
       (effects (font (size 1.27 1.27)) hide)
     )
-    (property "Voltage" "80V" (at 101.6 45.72 0)
+    (property "Voltage" "50V" (at 101.6 45.72 0)
       (effects (font (size 1.27 1.27)))
     )
     (property "R" "45 mOhm" (at 101.6 43.18 0)
       (effects (font (size 1.27 1.27)))
+    )
+    (property "MFR" "865060657011" (at 101.6 52.07 90)
+      (effects (font (size 1.27 1.27)) hide)
     )
     (pin "1")
@@
       (effects (font (size 1.27 1.27)) (justify left))
     )
-    (property "Footprint" "" (at 58.42 113.03 0)
+    (property "Footprint" "Connector_Molex:Molex_Mini-Fit_Jr_5566-04A2_2x02_P4.20mm_Vertical" (at 58.42 113.03 0)
       (effects (font (size 1.27 1.27)) hide)
     )
@@
       (effects (font (size 1.27 1.27)) (justify left))
     )
-    (property "Footprint" "" (at 144.78 45.72 0)
+    (property "Footprint" "Capacitor_SMD:C_0603_1608Metric_Pad1.08x0.95mm_HandSolder" (at 144.78 45.72 0)
       (effects (font (size 1.27 1.27)) hide)
     )
@@
         (path "/8b56e416-62b3-4f2a-b418-32bd641a0e6c"
           (reference "#PWR020") (unit 1)
-        )
-      )
-    )
-  )
-  (symbol (lib_id "Device:D_Schottky") (at 58.42 52.07 270) (unit 1)
-    (in_bom yes) (on_board yes) (dnp no)
-    (property "Reference" "D8" (at 55.88 49.53 0)
-      (effects (font (size 1.27 1.27)) (justify left))
-    )
-    (property "Value" "SMBJ54A" (at 60.96 48.26 0)
-      (effects (font (size 1.27 1.27)) (justify left))
-    )
-    (property "Footprint" "" (at 58.42 52.07 0)
-      (effects (font (size 1.27 1.27)) hide)
-    )
-    (property "Datasheet" "~" (at 58.42 52.07 0)
-      (effects (font (size 1.27 1.27)) hide)
-    )
-    (pin "1")
-    (pin "2")
-    (instances
-      (project "Robourt"
-        (path "/87ede840-4957-4951-b25a-c132e7988ddc/c536fa3c-09d4-4c8c-ac7c-935d025d1d35"
-          (reference "D8") (unit 1)
-        )
-        (path "/87ede840-4957-4951-b25a-c132e7988ddc/26d05491-2800-4f91-9931-a85caf6c3ce4"
-          (reference "D7") (unit 1)
-        )
-        (path "/87ede840-4957-4951-b25a-c132e7988ddc/807609e6-6522-4206-8069-5cb73bf05af8"
-          (reference "D9") (unit 1)
-        )
-      )
-      (project "driver_stepperLucas"
-        (path "/8b56e416-62b3-4f2a-b418-32bd641a0e6c"
-          (reference "D201") (unit 1)
         )
       )
@@
       (effects (font (size 1.27 1.27)) (justify left))
     )
-    (property "Footprint" "" (at 70.8152 55.88 0)
+    (property "Footprint" "Capacitor_SMD:CP_Elec_10x10.5" (at 70.8152 55.88 0)
       (effects (font (size 1.27 1.27)) hide)
     )
@@
       (effects (font (size 1.27 1.27)) hide)
     )
-    (property "Voltage" "80V" (at 69.85 45.72 0)
+    (property "Voltage" "50V" (at 69.85 45.72 0)
       (effects (font (size 1.27 1.27)))
     )
     (property "R" "45 mOhm" (at 69.85 43.18 0)
       (effects (font (size 1.27 1.27)))
+    )
+    (property "MFR" "865060657011" (at 69.85 52.07 90)
+      (effects (font (size 1.27 1.27)) hide)
     )
     (pin "1")
@@
       (effects (font (size 1.27 1.27)) (justify left))
     )
-    (property "Footprint" "" (at 82.2452 55.88 0)
+    (property "Footprint" "Capacitor_SMD:CP_Elec_10x10.5" (at 82.2452 55.88 0)
       (effects (font (size 1.27 1.27)) hide)
     )
@@
       (effects (font (size 1.27 1.27)) hide)
     )
-    (property "Voltage" "80V" (at 81.28 45.72 0)
+    (property "Voltage" "50V" (at 81.28 45.72 0)
       (effects (font (size 1.27 1.27)))
     )
     (property "R" "45 mOhm" (at 81.28 43.18 0)
       (effects (font (size 1.27 1.27)))
+    )
+    (property "MFR" "865060657011" (at 81.28 52.07 90)
+      (effects (font (size 1.27 1.27)) hide)
     )
     (pin "1")
@@
       (effects (font (size 1.27 1.27)) (justify right))
     )
-    (property "Footprint" "" (at 235.458 101.6 90)
+    (property "Footprint" "Resistor_SMD:R_2512_6332Metric_Pad1.40x3.35mm_HandSolder" (at 235.458 101.6 90)
       (effects (font (size 1.27 1.27)) hide)
     )
@@
       (effects (font (size 1.27 1.27)) (justify left))
     )
-    (property "Footprint" "" (at 235.458 36.83 90)
-      (effects (font (size 1.27 1.27)) hide)
-    )
+    (property "Footprint" "Resistor_SMD:R_2512_6332Metric_Pad1.40x3.35mm_HandSolder" (at 235.458 36.83 90)
+      (effects (font (size 1.27 1.27)) hide)
+    )

Commit message: pulled last changes from charlotte
Connections:
- net SG_TST: no longer names the net of U3.27 (SG_TST)
- net STANDALONE_MODE: no longer names the net of U3.26 (ST_ALONE)
- no-connect marks 0 -> 2
Changed lines of the file:
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@@
   (junction (at 233.68 119.38) (diameter 0) (color 0 0 0 0)
   )
+  (no_connect (at 152.4 91.44))
+  (no_connect (at 152.4 93.98))
   (wire (pts (xy 236.22 29.21) (xy 233.68 29.21))
     (stroke (width 0) (type default))
@@
     (effects (font (size 1.27 1.27)) (justify left))
   )
-  (hierarchical_label "STANDALONE_MODE" (shape input) (at 152.4 93.98 0) (fields_autoplaced)
-    (effects (font (size 1.27 1.27)) (justify left))
-  )
   (hierarchical_label "SCK" (shape input) (at 101.6 104.14 180) (fields_autoplaced)
     (effects (font (size 1.27 1.27)) (justify right))
@@
     (effects (font (size 1.27 1.27)) (justify right))
   )
-  (hierarchical_label "SG_TST" (shape input) (at 152.4 91.44 0) (fields_autoplaced)
-    (effects (font (size 1.27 1.27)) (justify left))
-  )
   (symbol (lib_name "SQJ504EP-T1_GE3_1") (lib_id "SQJ504EP-T1_GE3:SQJ504EP-T1_GE3") (at 224.79 124.46 180) (unit 1)

Commit message: update pcb
Parts:
- removed C27, C28: 150u, Capacitor_SMD:CP_Elec_10x10.5, symbol Device:C_Polarized
- added C203: 10u, Capacitor_SMD:C_2220_5750Metric, symbol Device:C_Small
- C201: renamed from C23; footprint Capacitor_SMD:C_0603_1608Metric_Pad1.08x0.95mm_HandSolder -> Capacitor_SMD:C_0402_1005Metric
- C202: renamed from C24; footprint Capacitor_SMD:C_0603_1608Metric_Pad1.08x0.95mm_HandSolder -> Capacitor_SMD:C_0402_1005Metric
- C206: renamed from C50; footprint Capacitor_SMD:C_0603_1608Metric_Pad1.08x0.95mm_HandSolder -> Capacitor_SMD:C_0402_1005Metric
- C207: renamed from C29; footprint Capacitor_SMD:C_0603_1608Metric_Pad1.08x0.95mm_HandSolder -> Capacitor_SMD:C_0402_1005Metric
- C208: renamed from C30; footprint Capacitor_SMD:C_0603_1608Metric_Pad1.08x0.95mm_HandSolder -> Capacitor_SMD:C_0402_1005Metric
- C209: renamed from C31; footprint Capacitor_SMD:C_0603_1608Metric_Pad1.08x0.95mm_HandSolder -> Capacitor_SMD:C_0402_1005Metric
- J201: renamed from J8; footprint Connector_Molex:Molex_Mini-Fit_Jr_5566-04A2_2x02_P4.20mm_Vertical -> Connector_Molex:Molex_Mini-Fit_Jr_5566-04A_2x02_P4.20mm_Vertical
- Q201: renamed from Q1; footprint Mosfet:SQJ968EPT1GE3 -> SQJ968EPT1GE3
- Q202: renamed from Q6; footprint Mosfet:SQJ968EPT1GE3 -> SQJ968EPT1GE3
- Q203: renamed from Q7; footprint Mosfet:SQJ968EPT1GE3 -> SQJ968EPT1GE3
- Q204: renamed from Q8; footprint Mosfet:SQJ968EPT1GE3 -> SQJ968EPT1GE3
- R201: renamed from R26; footprint Resistor_SMD:R_2512_6332Metric_Pad1.40x3.35mm_HandSolder -> Resistor_SMD:R_2512_6332Metric
- R202: renamed from R27; footprint Resistor_SMD:R_2512_6332Metric_Pad1.40x3.35mm_HandSolder -> Resistor_SMD:R_2512_6332Metric
- R203: renamed from R24; footprint Resistor_SMD:R_0603_1608Metric_Pad0.98x0.95mm_HandSolder -> Resistor_SMD:R_0402_1005Metric
- R204: renamed from R9; footprint Resistor_SMD:R_0603_1608Metric_Pad0.98x0.95mm_HandSolder -> Resistor_SMD:R_0402_1005Metric
- renumbered C25 to C204, C26 to C205, U3 to U201
Connections:
- net ENN is gone; now on net GND: U201.15 (ENN)
- net B1: now also Q202.4 (G2); no longer Q202.6 (D2)
- net GND: now also C203.2
- net HB1: now also Q202.6 (D2); no longer Q202.4 (G2)
- net Vdc: now also Q202.1 (S1), C203.1; no longer Q202.3 (S2)
- net at Q204.1 (S1), R202.1, R204.1: now also Q202.3 (S2); no longer Q202.1 (S1)
- net CLK: no longer names the net of U201.16 (CLK)
- net DIR: no longer names the net of U201.30 (DIR)
- net STEP: no longer names the net of U201.31 (STEP)
- no-connect marks 2 -> 5

Commit message: PCB changes
Connections:
- net B1: now also Q202.6 (D2); no longer Q202.4 (G2)
- net HB1: now also Q202.4 (G2); no longer Q202.6 (D2)
- net S: now reaches Q202.3 (S2), Q204.1 (S1), R202.1, R204.1

Commit message: lib working for all + PCB progress
Parts:
- Q201, Q202, Q203, Q204: footprint SQJ968EPT1GE3 -> Mosfet:SQJ968EPT1GE3
Changed lines of the file:
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@@
       (effects (font (size 1.27 1.27)))
     )
-    (property "Footprint" "SQJ968EPT1GE3" (at 205.74 29.54 0)
+    (property "Footprint" "Mosfet:SQJ968EPT1GE3" (at 205.74 29.54 0)
       (effects (font (size 1.27 1.27)) (justify left top) hide)
     )
@@
       (effects (font (size 1.27 1.27)))
     )
-    (property "Footprint" "SQJ968EPT1GE3" (at 266.7 214.3 0)
+    (property "Footprint" "Mosfet:SQJ968EPT1GE3" (at 266.7 214.3 0)
       (effects (font (size 1.27 1.27)) (justify left top) hide)
     )
@@
       (effects (font (size 1.27 1.27)))
     )
-    (property "Footprint" "SQJ968EPT1GE3" (at 262.89 149.53 0)
+    (property "Footprint" "Mosfet:SQJ968EPT1GE3" (at 262.89 149.53 0)
       (effects (font (size 1.27 1.27)) (justify left top) hide)
     )
@@
       (effects (font (size 1.27 1.27)))
     )
-    (property "Footprint" "SQJ968EPT1GE3" (at 201.93 149.53 0)
-      (effects (font (size 1.27 1.27)) (justify left top) hide)
-    )
+    (property "Footprint" "Mosfet:SQJ968EPT1GE3" (at 201.93 149.53 0)
+      (effects (font (size 1.27 1.27)) (justify left top) hide)
+    )
