File: Kicad/Eve/Robourt.kicad_sch (KiCad schematic)
At the start: 24 parts, among them IC1 STM32U535RET6, J2 Conn_01x02, J4 Conn_01x03, J5 Conn_01x03, J6 Conn_02x20_Odd_Even, J9 Conn_ST_STDC14, SW1 SW_Push, Y2 Crystal

Commit message: empreinte 13/11
Parts:
- C37, C8: value 10pF -> 10p; footprint (none) -> Capacitor_SMD:C_0603_1608Metric_Pad1.08x0.95mm_HandSolder
- H1, H2, H3, H4: footprint MountingHole:MountingHole_2.7mm_Pad_Via -> (none)
- IC1: footprint QFP50P1200X1200X160-64N -> STM32U535RET6:QFP50P1200X1200X160-64N
- J9: footprint Connector_PinHeader_1.27mm:PinHeader_2x07_P1.27mm_Vertical_SMD -> (none)
- R17: footprint (none) -> Resistor_SMD:R_0603_1608Metric_Pad0.98x0.95mm_HandSolder
Changed lines of the file:
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@@
       (effects (font (size 1.27 1.27)))
     )
-    (property "Footprint" "QFP50P1200X1200X160-64N" (at 114.3 275.26 0)
+    (property "Footprint" "STM32U535RET6:QFP50P1200X1200X160-64N" (at 114.3 275.26 0)
       (effects (font (size 1.27 1.27)) (justify left top) hide)
     )
@@
       (effects (font (size 1.27 1.27)) (justify left) hide)
     )
-    (property "Footprint" "MountingHole:MountingHole_2.7mm_Pad_Via" (at 245.11 39.37 0)
+    (property "Footprint" "" (at 245.11 39.37 0)
       (effects (font (size 1.27 1.27)) hide)
     )
@@
       (effects (font (size 1.27 1.27)) (justify left) hide)
     )
-    (property "Footprint" "MountingHole:MountingHole_2.7mm_Pad_Via" (at 224.79 39.37 0)
+    (property "Footprint" "" (at 224.79 39.37 0)
       (effects (font (size 1.27 1.27)) hide)
     )
@@
       (effects (font (size 1.27 1.27)) (justify right))
     )
-    (property "Value" "10pF" (at 233.68 115.57 90)
+    (property "Value" "10p" (at 233.68 115.57 90)
       (effects (font (size 1.27 1.27)) (justify right))
     )
-    (property "Footprint" "" (at 232.41 109.22 0)
+    (property "Footprint" "Capacitor_SMD:C_0603_1608Metric_Pad1.08x0.95mm_HandSolder" (at 232.41 109.22 0)
       (effects (font (size 1.27 1.27)) hide)
     )
@@
       (effects (font (size 1.27 1.27)))
     )
-    (property "Footprint" "" (at 246.38 110.998 90)
+    (property "Footprint" "Resistor_SMD:R_0603_1608Metric_Pad0.98x0.95mm_HandSolder" (at 246.38 110.998 90)
       (effects (font (size 1.27 1.27)) hide)
     )
@@
       (effects (font (size 1.27 1.27)) (justify left) hide)
     )
-    (property "Footprint" "MountingHole:MountingHole_2.7mm_Pad_Via" (at 256.54 39.37 0)
+    (property "Footprint" "" (at 256.54 39.37 0)
       (effects (font (size 1.27 1.27)) hide)
     )
@@
       (effects (font (size 1.27 1.27)) (justify right))
     )
-    (property "Footprint" "Connector_PinHeader_1.27mm:PinHeader_2x07_P1.27mm_Vertical_SMD" (at 367.03 165.1 0)
+    (property "Footprint" "" (at 367.03 165.1 0)
       (effects (font (size 1.27 1.27)) hide)
     )
@@
   (symbol (lib_id "Device:C_Small") (at 232.41 96.52 270) (unit 1)
     (in_bom yes) (on_board yes) (dnp no) (fields_autoplaced)
-    (property "Reference" "C8" (at 232.4036 90.17 90)
-      (effects (font (size 1.27 1.27)))
-    )
-    (property "Value" "10pF" (at 232.4036 92.71 90)
-      (effects (font (size 1.27 1.27)))
-    )
-    (property "Footprint" "" (at 232.41 96.52 0)
+    (property "Reference" "C8" (at 232.4036 91.44 90)
+      (effects (font (size 1.27 1.27)))
+    )
+    (property "Value" "10p" (at 232.4036 93.98 90)
+      (effects (font (size 1.27 1.27)))
+    )
+    (property "Footprint" "Capacitor_SMD:C_0603_1608Metric_Pad1.08x0.95mm_HandSolder" (at 232.41 96.52 0)
       (effects (font (size 1.27 1.27)) hide)
     )
@@
       (effects (font (size 1.27 1.27)) (justify left) hide)
     )
-    (property "Footprint" "MountingHole:MountingHole_2.7mm_Pad_Via" (at 234.95 39.37 0)
-      (effects (font (size 1.27 1.27)) hide)
-    )
+    (property "Footprint" "" (at 234.95 39.37 0)
+      (effects (font (size 1.27 1.27)) hide)
+    )

Commit message: pulled main and started routing
Parts:
- H1, H2, H3, H4: footprint (none) -> MountingHole:MountingHole_3.2mm_M3_Pad_Via
- J2: footprint Connector_JST:JST_XH_B2B-XH-A_1x02_P2.50mm_Vertical -> Connector_AMASS:AMASS_XT60-F_1x02_P7.20mm_Vertical
- J4, J5: footprint (none) -> Connector_JST:JST_XH_B3B-XH-A_1x03_P2.50mm_Vertical
- J9: footprint (none) -> Connector_PinHeader_1.27mm:PinHeader_2x07_P1.27mm_Vertical_SMD
Changed lines of the file:
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@@
       (effects (font (size 1.27 1.27)) (justify left) hide)
     )
-    (property "Footprint" "" (at 245.11 39.37 0)
+    (property "Footprint" "MountingHole:MountingHole_3.2mm_M3_Pad_Via" (at 245.11 39.37 0)
       (effects (font (size 1.27 1.27)) hide)
     )
@@
       (effects (font (size 1.27 1.27)) (justify left))
     )
-    (property "Footprint" "" (at 255.27 210.82 0)
+    (property "Footprint" "Connector_JST:JST_XH_B3B-XH-A_1x03_P2.50mm_Vertical" (at 255.27 210.82 0)
       (effects (font (size 1.27 1.27)) hide)
     )
@@
       (effects (font (size 1.27 1.27)) (justify left) hide)
     )
-    (property "Footprint" "" (at 224.79 39.37 0)
+    (property "Footprint" "MountingHole:MountingHole_3.2mm_M3_Pad_Via" (at 224.79 39.37 0)
       (effects (font (size 1.27 1.27)) hide)
     )
@@
       (effects (font (size 1.27 1.27)) (justify left))
     )
-    (property "Footprint" "" (at 255.27 194.31 0)
+    (property "Footprint" "Connector_JST:JST_XH_B3B-XH-A_1x03_P2.50mm_Vertical" (at 255.27 194.31 0)
       (effects (font (size 1.27 1.27)) hide)
     )
@@
       (effects (font (size 1.27 1.27)) (justify left) hide)
     )
-    (property "Footprint" "" (at 256.54 39.37 0)
+    (property "Footprint" "MountingHole:MountingHole_3.2mm_M3_Pad_Via" (at 256.54 39.37 0)
       (effects (font (size 1.27 1.27)) hide)
     )
@@
       (effects (font (size 1.27 1.27)) (justify right))
     )
-    (property "Footprint" "" (at 367.03 165.1 0)
+    (property "Footprint" "Connector_PinHeader_1.27mm:PinHeader_2x07_P1.27mm_Vertical_SMD" (at 367.03 165.1 0)
       (effects (font (size 1.27 1.27)) hide)
     )
@@
       (effects (font (size 1.27 1.27)))
     )
-    (property "Footprint" "Connector_JST:JST_XH_B2B-XH-A_1x02_P2.50mm_Vertical" (at 261.62 173.99 0)
+    (property "Footprint" "Connector_AMASS:AMASS_XT60-F_1x02_P7.20mm_Vertical" (at 261.62 173.99 0)
       (effects (font (size 1.27 1.27)) hide)
     )
@@
       (effects (font (size 1.27 1.27)) (justify left) hide)
     )
-    (property "Footprint" "" (at 234.95 39.37 0)
-      (effects (font (size 1.27 1.27)) hide)
-    )
+    (property "Footprint" "MountingHole:MountingHole_3.2mm_M3_Pad_Via" (at 234.95 39.37 0)
+      (effects (font (size 1.27 1.27)) hide)
+    )

Commit message: pulled last changes from charlotte
Connections:
- no-connect marks 72 -> 66
Other:
- sheet driver_stepper ports: added none; removed SG_TST, STANDALONE_MODE
- sheet driver_stepper1 ports: added none; removed SG_TST, STANDALONE_MODE
- sheet driver_stepper2 ports: added none; removed SG_TST, STANDALONE_MODE
Changed lines of the file:
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@@
   (no_connect (at 347.98 234.95))
   (no_connect (at 95.25 172.72))
-  (no_connect (at 135.89 82.55))
   (no_connect (at 365.76 222.25))
   (no_connect (at 90.17 251.46))
@@
   (no_connect (at 92.71 172.72))
   (no_connect (at 105.41 251.46))
-  (no_connect (at 80.01 62.23))
   (no_connect (at 118.11 231.14))
   (no_connect (at 85.09 172.72))
@@
   (no_connect (at 118.11 226.06))
   (no_connect (at 353.06 234.95))
-  (no_connect (at 27.94 73.66))
   (no_connect (at 92.71 251.46))
   (no_connect (at 64.77 195.58))
   (no_connect (at 354.33 170.18))
   (no_connect (at 105.41 172.72))
-  (no_connect (at 80.01 67.31))
   (no_connect (at 373.38 234.95))
   (no_connect (at 350.52 234.95))
@@
   (no_connect (at 27.94 55.88))
   (no_connect (at 64.77 233.68))
-  (no_connect (at 135.89 78.74))
   (no_connect (at 118.11 233.68))
   (no_connect (at 353.06 222.25))
@@
   (no_connect (at 370.84 222.25))
   (no_connect (at 354.33 165.1))
-  (no_connect (at 27.94 80.01))
   (no_connect (at 107.95 172.72))
   (wire (pts (xy 341.63 160.02) (xy 354.33 160.02))
@@
       (effects (font (size 1.27 1.27)) (justify left))
     )
-    (pin "STANDALONE_MODE" input (at 27.94 80.01 180)
-      (effects (font (size 1.27 1.27)) (justify left))
-    )
-    (pin "SG_TST" input (at 27.94 73.66 180)
-      (effects (font (size 1.27 1.27)) (justify left))
-    )
     (pin "SCK" input (at 33.02 114.3 270)
       (effects (font (size 1.27 1.27)) (justify left))
@@
       (effects (font (size 1.27 1.27)) (justify right))
     )
-    (pin "STANDALONE_MODE" input (at 135.89 82.55 180)
-      (effects (font (size 1.27 1.27)) (justify left))
-    )
-    (pin "SG_TST" input (at 135.89 78.74 180)
-      (effects (font (size 1.27 1.27)) (justify left))
-    )
     (pin "SCK" input (at 139.7 114.3 270)
       (effects (font (size 1.27 1.27)) (justify left))
@@
       (effects (font (size 1.27 1.27)) (justify left))
     )
-    (pin "SG_TST" input (at 80.01 62.23 180)
-      (effects (font (size 1.27 1.27)) (justify left))
-    )
-    (pin "STANDALONE_MODE" input (at 80.01 67.31 180)
-      (effects (font (size 1.27 1.27)) (justify left))
-    )

Commit message: update pcb
Parts:
- removed C3: 100n, Capacitor_SMD:C_0603_1608Metric_Pad1.08x0.95mm_HandSolder, symbol Device:C
- removed SW1: SW_Push, Button_Switch_SMD:SW_SPST_B3U-1000P, symbol Switch:SW_Push
- added C103, C104, C109, C110, C112, C113, C114, C115, C118, C119, C120, C121: 100n, Capacitor_SMD:C_0402_1005Metric, symbol Device:C_Small
- added C?: 4.7u, Capacitor_SMD:C_0402_1005Metric, symbol Device:C
- added C? (x2): 100n, Capacitor_SMD:C_0402_1005Metric, symbol Device:C
- added D? (x3): LED, LED_SMD:LED_0603_1608Metric, symbol Device:LED
- added J102, J103, J104, J105, J106, J107, J111, J112, J113, J114: Conn_01x02, Connector_JST:JST_XH_B2B-XH-A_1x02_P2.50mm_Vertical, symbol Connector_Generic:Conn_01x02
- added Q101: NMOS, Package_TO_SOT_SMD:SOT-23, symbol Simulation_SPICE:NMOS
- added R101, R102, R110, R111, R115, R116, R117, R118, R125, R126, R127, R128: 100k, Resistor_SMD:R_0402_1005Metric, symbol Device:R_Small
- added R103, R104, R112, R113, R120, R121, R122, R123, R129, R130, R131, R132: 1k, Resistor_SMD:R_0402_1005Metric, symbol Device:R_Small
- added R107: 22, Resistor_SMD:R_0402_1005Metric, symbol Device:R_Small
- added R108: 10k, Resistor_SMD:R_0402_1005Metric, symbol Device:R_Small
- added R? (x3): 390, Resistor_SMD:R_0402_1005Metric, symbol Device:R
- added SW? (x4): SW_Push, Button_Switch_SMD:SW_SPST_B3U-1000P, symbol Switch:SW_Push
- C116: renamed from C8; footprint Capacitor_SMD:C_0603_1608Metric_Pad1.08x0.95mm_HandSolder -> Capacitor_SMD:C_0402_1005Metric
- C117: renamed from C37; footprint Capacitor_SMD:C_0603_1608Metric_Pad1.08x0.95mm_HandSolder -> Capacitor_SMD:C_0402_1005Metric
- C?: renamed from C5; footprint Capacitor_SMD:C_0603_1608Metric_Pad1.08x0.95mm_HandSolder -> Capacitor_SMD:C_0402_1005Metric
- C?: renamed from C6; footprint Capacitor_SMD:C_0603_1608Metric_Pad1.08x0.95mm_HandSolder -> Capacitor_SMD:C_0402_1005Metric
- C?: renamed from C7; footprint Capacitor_SMD:C_0603_1608Metric_Pad1.08x0.95mm_HandSolder -> Capacitor_SMD:C_0402_1005Metric
- C?: renamed from C4; footprint Capacitor_SMD:C_0603_1608Metric_Pad1.08x0.95mm_HandSolder -> Capacitor_SMD:C_0402_1005Metric
- D105, D?: renamed from D2; footprint LED_SMD:LED_0603_1608Metric_Pad1.05x0.95mm_HandSolder -> LED_SMD:LED_0603_1608Metric
- J?: renamed from J6; footprint Connector_PinHeader_2.54mm:PinHeader_2x20_P2.54mm_Vertical -> Connector_PinSocket_2.54mm:PinSocket_2x20_P2.54mm_Horizontal
- R119: renamed from R3; footprint Resistor_SMD:R_0603_1608Metric_Pad0.98x0.95mm_HandSolder -> Resistor_SMD:R_0402_1005Metric
- R124: renamed from R17; footprint Resistor_SMD:R_0603_1608Metric_Pad0.98x0.95mm_HandSolder -> Resistor_SMD:R_0402_1005Metric
- R?: renamed from R3; value 1k -> 390; footprint Resistor_SMD:R_0603_1608Metric_Pad0.98x0.95mm_HandSolder -> Resistor_SMD:R_0402_1005Metric
- renumbered H3 to H?, H1 to H?, H4 to H?, H2 to H?, IC1 to IC101, J4 to J108, J5 to J109, J2 to J110, J9 to J?, Y2 to Y101
Connections:
- net GPIO_DIR2 is gone; now on net GPIO_CSN1: IC101.39 (PC8)
- net GPIO_DIR3 is gone; now on net GPIO_CSN3: IC101.37 (PC6)
- net GPIO_STEP3 is gone; now on net GPIO_CSN2: IC101.38 (PC7)
- net +3.3V: now also IC101.1 (VBAT), C?.1, C?.1, R101.1, R102.1, R110.1, R111.1, R115.1, R116.1, R117.1, R118.1, R125.1, R126.1, R127.1, R128.1
- net 5.1V: now also J102.1 (Pin_1), J103.1 (Pin_1)
- net GND: now also IC101.60 (PH3-BOOT0), C103.2, C104.2, C109.2, C110.2, C112.2, C113.2, C114.2, C115.2, C118.2, C119.2, C120.2, C121.2, C?.2, C?.2, C?.2, J104.2 (Pin_2), J105.2 (Pin_2), J106.2 (Pin_2), J107.2 (Pin_2), J111.2 (Pin_2), J112.2 (Pin_2), J113.2 (Pin_2), J114.2 (Pin_2), Q101.3 (S), R108.2, R?.2, R?.2, R?.2, SW?.2, SW?.2, SW?.2, SW?.2
- net GPIO_CSN1: no longer IC101.45 (PA12)
- net GPIO_CSN2: no longer IC101.44 (PA11)
- net GPIO_CSN3: no longer IC101.43 (PA10)
- net NRST: now also C103.1, R101.2, R103.1
- net SCK: now also IC101.34 (PB13); no longer IC101.29 (PB10)
- net SPI2_MISO: now also IC101.35 (PB14); no longer IC101.10 (PC2)
- net SPI2_MOSI: now also IC101.36 (PB15); no longer IC101.11 (PC3)
- net UART4_RX: now also IC101.15 (PA1); no longer IC101.52 (PC11)
- net USART1_TX: now also J108.1 (Pin_1)
- net FDC_1: now reaches IC101.20 (PA4)
- net FDC_1: now also C112.1, R115.2, R120.1
- net FDC_2: now reaches IC101.21 (PA5)
- net FDC_2: now also C113.1, R116.2, R121.1
- net FDC_3: now reaches IC101.22 (PA6)
- net FDC_3: now also C114.1, R117.2, R122.1
- net FDC_5: now reaches IC101.24 (PC4)
- net FDC_5: now also C118.1, R125.2, R129.1
- net FDC_6: now reaches IC101.25 (PC5)
- net FDC_6: now also C119.1, R126.2, R130.1
- net FDC_7: now reaches IC101.26 (PB0)
- net FDC_7: now also C120.1, R127.2, R131.1
- net FDC_8: now reaches IC101.27 (PB1)
- net FDC_8: now also C121.1, R128.2, R132.1
- net Vcap: now reaches IC101.30 (VCAP)
- net Vcap: now also C?.1
- net USR_BTN_3: now reaches IC101.51 (PC10)
- net USR_BTN_3: now also C110.1, R111.2, R113.1
- net SYS_JTDO-SWO: now reaches IC101.55 (PB3)
- net SYS_JTDO-SWO: now also J?.8 (JTDO/SWO)
- net PWM_FAN: now reaches IC101.62 (PB9)
- net PWM_FAN: now also R107.1
- net GPIO_DIR1 renamed USR_LED_4
- net USR_LED_4: now also D?.2 (A)
- net GPIO_STEP1 renamed USR_LED_3
- net USR_LED_3: now also D?.2 (A)
- net GPIO_STEP2: no longer names the net of IC101.40 (PC9)
- net Test_LED renamed USR_LED_1
- net USR_LED_1: now also IC101.44 (PA11); no longer IC101.15 (PA1)
- net UART5_TX renamed USR_BTN_1
- net USR_BTN_1: now also C109.1, R110.2, R112.1
- net USART3_TX renamed FDC_4
- net FDC_4: now also C115.1, R118.2, R123.1; no longer J108.1 (Pin_1)
- new net: D?.1 (K), R?.1 (x3)
- new net: R104.2, SW?.1
- new net: J102.2 (Pin_2), J103.2 (Pin_2), Q101.1 (D)
- new net: Q101.2 (G), R107.2, R108.1
- new net: J113.1 (Pin_1), R131.2
- new net: R103.2, SW?.1
- new net: J107.1 (Pin_1), R123.2
- new net: J105.1 (Pin_1), R121.2
- new net: J114.1 (Pin_1), R132.2
- new net: J106.1 (Pin_1), R122.2
- new net: J112.1 (Pin_1), R130.2
- new net: R113.2, SW?.1
- new net: R112.2, SW?.1
- new net: J104.1 (Pin_1), R120.2
- new net: J111.1 (Pin_1), R129.2
- new net USR_BTN_2: C104.1, IC101.52 (PC11), R102.2, R104.1
- new net USR_LED_2: D?.2 (A), IC101.43 (PA10)
- no-connect marks 66 -> 48
Other:
- sheet driver_stepper ports: added none; removed CLK, DIR, ENN, STEP
- sheet driver_stepper1 ports: added none; removed CLK, DIR, ENN, STEP
- sheet driver_stepper2 ports: added none; removed CLK, DIR, ENN, STEP
- note added: "USART 1 : XL430 LPUART 1 : Rpi UART 4 : ST-Link"
- moved on the sheet: C116, C117, C?, D105, D?, H?, IC101, J108, J109, J110, J?, R119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
