File: Kicad/Eve/Robourt.kicad_sch (KiCad schematic)
At the start: 84 parts, among them IC101 STM32U535RET6, J102 Conn_01x02, J103 Conn_01x02, J104 Conn_01x02, J105 Conn_01x02, J106 Conn_01x02, J107 Conn_01x02, J108 Conn_01x03, J109 Conn_01x03, J110 Conn_01x02, J111 Conn_01x02, J112 Conn_01x02, J113 Conn_01x02, J114 Conn_01x02, Q101 NMOS, Y101 Crystal

Commit message: PCB changes
Parts:
- removed J104, J105, J106, J107, J111, J112, J113, J114: Conn_01x02, Connector_JST:JST_XH_B2B-XH-A_1x02_P2.50mm_Vertical, symbol Connector_Generic:Conn_01x02
- added J1: Conn_02x08_Odd_Even, Connector_PinSocket_2.54mm:PinSocket_2x08_P2.54mm_Vertical_SMD, symbol Connector_Generic:Conn_02x08_Odd_Even
Changed lines of the file:
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@@
     )
   )
-  (symbol (lib_id "Connector_Generic:Conn_01x02") (at 264.16 237.49 0) (unit 1)
-    (in_bom yes) (on_board yes) (dnp no) (fields_autoplaced)
-    (property "Reference" "J113" (at 266.7 237.49 0)
-      (effects (font (size 1.27 1.27)) (justify left))
-    )
-    (property "Value" "Conn_01x02" (at 266.7 240.03 0)
-      (effects (font (size 1.27 1.27)) (justify left))
-    )
-    (property "Footprint" "Connector_JST:JST_XH_B2B-XH-A_1x02_P2.50mm_Vertical" (at 264.16 237.49 0)
-      (effects (font (size 1.27 1.27)) hide)
-    )
-    (property "Datasheet" "~" (at 264.16 237.49 0)
-      (effects (font (size 1.27 1.27)) hide)
-    )
-    (pin "2")
-    (pin "1")
-    (instances
-      (project "Robourt"
-        (path "/87ede840-4957-4951-b25a-c132e7988ddc"
-          (reference "J113") (unit 1)
-        )
-      )
-    )
-  )
   (symbol (lib_id "power:+3.3V") (at 96.52 113.03 270) (unit 1)
     (in_bom yes) (on_board yes) (dnp no) (fields_autoplaced)
@@
     )
   )
+  (symbol (lib_id "Connector_Generic:Conn_02x08_Odd_Even") (at 226.06 158.75 0) (unit 1)
+    (in_bom yes) (on_board yes) (dnp no) (fields_autoplaced)
+    (property "Reference" "J1" (at 227.33 144.78 0)
+      (effects (font (size 1.27 1.27)))
+    )
+    (property "Value" "Conn_02x08_Odd_Even" (at 227.33 147.32 0)
+      (effects (font (size 1.27 1.27)))
+    )
+    (property "Footprint" "Connector_PinSocket_2.54mm:PinSocket_2x08_P2.54mm_Vertical_SMD" (at 226.06 158.75 0)
+      (effects (font (size 1.27 1.27)) hide)
+    )
+    (property "Datasheet" "~" (at 226.06 158.75 0)
+      (effects (font (size 1.27 1.27)) hide)
+    )
+    (pin "1")
+    (pin "11")
+    (pin "12")
+    (pin "6")
+    (pin "10")
+    (pin "9")
+    (pin "4")
+    (pin "5")
+    (pin "7")
+    (pin "15")
+    (pin "13")
+    (pin "8")
+    (pin "16")
+    (pin "14")
+    (pin "2")
+    (pin "3")
+    (instances
+      (project "Robourt"
+        (path "/87ede840-4957-4951-b25a-c132e7988ddc"
+          (reference "J1") (unit 1)
+        )
+      )
+    )
+  )
   (symbol (lib_id "power:PWR_FLAG") (at 378.46 31.75 0) (unit 1)
     (in_bom yes) (on_board yes) (dnp no)
@@
     )
   )
-  (symbol (lib_id "Connector_Generic:Conn_01x02") (at 264.16 266.7 0) (unit 1)
-    (in_bom yes) (on_board yes) (dnp no) (fields_autoplaced)
-    (property "Reference" "J114" (at 266.7 266.7 0)
-      (effects (font (size 1.27 1.27)) (justify left))
-    )
-    (property "Value" "Conn_01x02" (at 266.7 269.24 0)
-      (effects (font (size 1.27 1.27)) (justify left))
-    )
-    (property "Footprint" "Connector_JST:JST_XH_B2B-XH-A_1x02_P2.50mm_Vertical" (at 264.16 266.7 0)
-      (effects (font (size 1.27 1.27)) hide)
-    )
-    (property "Datasheet" "~" (at 264.16 266.7 0)
-      (effects (font (size 1.27 1.27)) hide)
-    )
-    (pin "2")
-    (pin "1")
-    (instances
-      (project "Robourt"
-        (path "/87ede840-4957-4951-b25a-c132e7988ddc"
-          (reference "J114") (unit 1)
-        )
-      )
-    )
-  )
   (symbol (lib_id "power:GND") (at 337.82 100.33 180) (unit 1)
     (in_bom yes) (on_board yes) (dnp no) (fields_autoplaced)
@@
     )
   )
-  (symbol (lib_id "Connector_Generic:Conn_01x02") (at 219.71 236.22 0) (unit 1)
-    (in_bom yes) (on_board yes) (dnp no) (fields_autoplaced)
-    (property "Reference" "J106" (at 222.25 236.22 0)
-      (effects (font (size 1.27 1.27)) (justify left))
-    )
-    (property "Value" "Conn_01x02" (at 222.25 238.76 0)
-      (effects (font (size 1.27 1.27)) (justify left))
-    )
-    (property "Footprint" "Connector_JST:JST_XH_B2B-XH-A_1x02_P2.50mm_Vertical" (at 219.71 236.22 0)
-      (effects (font (size 1.27 1.27)) hide)
-    )
-    (property "Datasheet" "~" (at 219.71 236.22 0)
-      (effects (font (size 1.27 1.27)) hide)
-    )
-    (pin "2")
-    (pin "1")
-    (instances
-      (project "Robourt"
-        (path "/87ede840-4957-4951-b25a-c132e7988ddc"
-          (reference "J106") (unit 1)
-        )
-      )
-    )
-  )
-  (symbol (lib_id "Connector_Generic:Conn_01x02") (at 219.71 265.43 0) (unit 1)
-    (in_bom yes) (on_board yes) (dnp no) (fields_autoplaced)
-    (property "Reference" "J107" (at 222.25 265.43 0)
-      (effects (font (size 1.27 1.27)) (justify left))
-    )
-    (property "Value" "Conn_01x02" (at 222.25 267.97 0)
-      (effects (font (size 1.27 1.27)) (justify left))
-    )
-    (property "Footprint" "Connector_JST:JST_XH_B2B-XH-A_1x02_P2.50mm_Vertical" (at 219.71 265.43 0)
-      (effects (font (size 1.27 1.27)) hide)
-    )
-    (property "Datasheet" "~" (at 219.71 265.43 0)
-      (effects (font (size 1.27 1.27)) hide)
-    )
-    (pin "2")
-    (pin "1")
-    (instances
-      (project "Robourt"
-        (path "/87ede840-4957-4951-b25a-c132e7988ddc"
-          (reference "J107") (unit 1)
-        )
-      )
-    )
-  )
   (symbol (lib_id "Device:C_Small") (at 220.98 45.72 270) (unit 1)
     (in_bom yes) (on_board yes) (dnp no)
@@
     )
   )
-  (symbol (lib_id "Connector_Generic:Conn_01x02") (at 219.71 207.01 0) (unit 1)
-    (in_bom yes) (on_board yes) (dnp no) (fields_autoplaced)
-    (property "Reference" "J105" (at 222.25 207.01 0)
-      (effects (font (size 1.27 1.27)) (justify left))
-    )
-    (property "Value" "Conn_01x02" (at 222.25 209.55 0)
-      (effects (font (size 1.27 1.27)) (justify left))
-    )
-    (property "Footprint" "Connector_JST:JST_XH_B2B-XH-A_1x02_P2.50mm_Vertical" (at 219.71 207.01 0)
-      (effects (font (size 1.27 1.27)) hide)
-    )
-    (property "Datasheet" "~" (at 219.71 207.01 0)
-      (effects (font (size 1.27 1.27)) hide)
-    )
-    (pin "2")
-    (pin "1")
-    (instances
-      (project "Robourt"
-        (path "/87ede840-4957-4951-b25a-c132e7988ddc"
-          (reference "J105") (unit 1)
-        )
-      )
-    )
-  )
   (symbol (lib_id "Device:R_Small") (at 254 234.95 90) (unit 1)
     (in_bom yes) (on_board yes) (dnp no)
@@
     )
   )
-  (symbol (lib_id "Connector_Generic:Conn_01x02") (at 219.71 177.8 0) (unit 1)
-    (in_bom yes) (on_board yes) (dnp no) (fields_autoplaced)
-    (property "Reference" "J104" (at 222.25 177.8 0)
-      (effects (font (size 1.27 1.27)) (justify left))
-    )
-    (property "Value" "Conn_01x02" (at 222.25 180.34 0)
-      (effects (font (size 1.27 1.27)) (justify left))
-    )
-    (property "Footprint" "Connector_JST:JST_XH_B2B-XH-A_1x02_P2.50mm_Vertical" (at 219.71 177.8 0)
-      (effects (font (size 1.27 1.27)) hide)
-    )
-    (property "Datasheet" "~" (at 219.71 177.8 0)
-      (effects (font (size 1.27 1.27)) hide)
-    )
-    (pin "2")
-    (pin "1")
-    (instances
-      (project "Robourt"
-        (path "/87ede840-4957-4951-b25a-c132e7988ddc"
-          (reference "J104") (unit 1)
-        )
-      )
-    )
-  )
   (symbol (lib_id "Mechanical:MountingHole_Pad") (at 351.79 149.86 0) (unit 1)
     (in_bom yes) (on_board yes) (dnp no)
@@
     )
   )
-  (symbol (lib_id "Connector_Generic:Conn_01x02") (at 264.16 207.01 0) (unit 1)
-    (in_bom yes) (on_board yes) (dnp no) (fields_autoplaced)
-    (property "Reference" "J112" (at 266.7 207.01 0)
-      (effects (font (size 1.27 1.27)) (justify left))
-    )
-    (property "Value" "Conn_01x02" (at 266.7 209.55 0)
-      (effects (font (size 1.27 1.27)) (justify left))
-    )
-    (property "Footprint" "Connector_JST:JST_XH_B2B-XH-A_1x02_P2.50mm_Vertical" (at 264.16 207.01 0)
-      (effects (font (size 1.27 1.27)) hide)
-    )
-    (property "Datasheet" "~" (at 264.16 207.01 0)
-      (effects (font (size 1.27 1.27)) hide)
-    )
-    (pin "2")
-    (pin "1")
-    (instances
-      (project "Robourt"
-        (path "/87ede840-4957-4951-b25a-c132e7988ddc"
-          (reference "J112") (unit 1)
-        )
-      )
-    )
-  )
   (symbol (lib_id "power:GND") (at 96.52 115.57 90) (unit 1)
     (in_bom yes) (on_board yes) (dnp no) (fields_autoplaced)
@@
         )
       )
-    )
-  )
-  (symbol (lib_id "Connector_Generic:Conn_01x02") (at 264.16 177.8 0) (unit 1)
-    (in_bom yes) (on_board yes) (dnp no) (fields_autoplaced)
-    (property "Reference" "J111" (at 266.7 177.8 0)
-      (effects (font (size 1.27 1.27)) (justify left))
-    )
-    (property "Value" "Conn_01x02" (at 266.7 180.34 0)
-      (effects (font (size 1.27 1.27)) (justify left))
-    )
-    (property "Footprint" "Connector_JST:JST_XH_B2B-XH-A_1x02_P2.50mm_Vertical" (at 264.16 177.8 0)
-      (effects (font (size 1.27 1.27)) hide)
-    )
-    (property "Datasheet" "~" (at 264.16 177.8 0)
-      (effects (font (size 1.27 1.27)) hide)
-    )
-    (pin "2")
-    (pin "1")
-    (instances
-      (project "Robourt"
-        (path "/87ede840-4957-4951-b25a-c132e7988ddc"
-          (reference "J111") (unit 1)
-        )
-      )

Commit message: lib working for all + PCB progress
Parts:
- J1: footprint Connector_PinSocket_2.54mm:PinSocket_2x08_P2.54mm_Vertical_SMD -> Connector_PinHeader_2.00mm:PinHeader_2x08_P2.00mm_Vertical_SMD
Changed lines of the file:
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@@
       (effects (font (size 1.27 1.27)))
     )
-    (property "Footprint" "Connector_PinSocket_2.54mm:PinSocket_2x08_P2.54mm_Vertical_SMD" (at 226.06 158.75 0)
+    (property "Footprint" "Connector_PinHeader_2.00mm:PinHeader_2x08_P2.00mm_Vertical_SMD" (at 226.06 158.75 0)
       (effects (font (size 1.27 1.27)) hide)
     )

Commit message: update 17/12
Connections:
- net GND: now also J1.10 (Pin_10), J1.12 (Pin_12), J1.14 (Pin_14), J1.16 (Pin_16), J1.2 (Pin_2), J1.4 (Pin_4), J1.6 (Pin_6), J1.8 (Pin_8)
- net FDC4: now reaches R123.2
- net FDC4: now also J1.7 (Pin_7)
- net FDC1: now reaches J1.1 (Pin_1)
- net FDC1: now also R120.2
- net FDC6: now reaches J1.11 (Pin_11)
- net FDC6: now also R130.2
- net FDC7: now reaches J1.13 (Pin_13)
- net FDC7: now also R131.2
- net FDC8: now reaches J1.15 (Pin_15)
- net FDC8: now also R132.2
- net FDC2: now reaches J1.3 (Pin_3)
- net FDC2: now also R121.2
- net FDC3: now reaches J1.5 (Pin_5)
- net FDC3: now also R122.2
- net FDC5: now reaches J1.9 (Pin_9)
- net FDC5: now also R129.2
Other:
- note added: "Capteur de fin de course"
- note added: "Ventilateur"
- moved on the sheet: C118, C119, C120, C121, J1, R125, R126, R127, R128, R129, R130, R131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

Commit message: update 18/12
Parts:
- R119: value 1k -> 4k
Changed lines of the file:
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@@
       (effects (font (size 1.27 1.27)) (justify left))
     )
-    (property "Value" "1k" (at 210.82 100.965 0)
+    (property "Value" "4k" (at 210.82 100.965 0)
       (effects (font (size 1.27 1.27)) (justify left))
     )
