File: Kicad/Eve/Robourt.kicad_sch (KiCad schematic)
At the start: 77 parts, among them IC101 STM32U535RET6, J1 Conn_02x08_Odd_Even, J102 Conn_01x02, J103 Conn_01x02, J108 Conn_01x03, J109 Conn_01x03, J110 Conn_01x02, Q101 NMOS, Y101 Crystal

Commit message: update PCB
Connections:
- net FDC_6: now also IC101.26 (PB0); no longer IC101.25 (PC5)
- net FDC_7: now also IC101.25 (PC5); no longer IC101.26 (PB0)

Commit message: Big PCB update errors remain
Connections:
- net USR_BTN_2: now also IC101.51 (PC10); no longer IC101.52 (PC11)
- net USR_BTN_3: now also IC101.52 (PC11); no longer IC101.51 (PC10)
- net USR_LED_1: now also IC101.41 (PA8); no longer IC101.44 (PA11)
- net USR_LED_2: now also IC101.42 (PA9); no longer IC101.43 (PA10)
- net USR_LED_3: now also IC101.43 (PA10); no longer IC101.42 (PA9)
- net USR_LED_4: now also IC101.44 (PA11); no longer IC101.41 (PA8)
Changed lines of the file:
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@@
     (effects (font (size 1.27 1.27)) (justify left bottom))
-  )
-  (label "USR_BTN_3" (at 83.82 78.74 270) (fields_autoplaced)
-    (effects (font (size 1.27 1.27)) (justify right bottom))
   )
   (label "USR_BTN_1" (at 151.13 137.16 0) (fields_autoplaced)
@@
     (effects (font (size 1 1)) (justify left bottom))
   )
-  (label "USR_BTN_2" (at 81.28 78.74 270) (fields_autoplaced)
-    (effects (font (size 1.27 1.27)) (justify right bottom))
-  )
-  (label "USR_LED_2" (at 109.22 125.73 180) (fields_autoplaced)
+  (label "USR_BTN_3" (at 81.28 78.74 270) (fields_autoplaced)
     (effects (font (size 1.27 1.27)) (justify right bottom))
   )
@@
     (effects (font (size 1.27 1.27)) (justify left bottom))
   )
+  (label "USR_LED_3" (at 109.22 125.73 180) (fields_autoplaced)
+    (effects (font (size 1.27 1.27)) (justify right bottom))
+  )
   (label "Vcap" (at 83.82 175.26 90) (fields_autoplaced)
     (effects (font (size 1.27 1.27)) (justify left bottom))
@@
     (effects (font (size 0.65 0.65)) (justify left bottom))
   )
+  (label "USR_BTN_2" (at 83.82 78.74 270) (fields_autoplaced)
+    (effects (font (size 1.27 1.27)) (justify right bottom))
+  )
   (label "FDC_2" (at 60.96 184.15 90) (fields_autoplaced)
     (effects (font (size 1.27 1.27)) (justify left bottom))
-  )
-  (label "USR_LED_3" (at 109.22 128.27 180) (fields_autoplaced)
-    (effects (font (size 1.27 1.27)) (justify right bottom))
   )
   (label "SYS_JTDO-SWO" (at 83.82 234.95 0) (fields_autoplaced)
     (effects (font (size 1 1)) (justify left bottom))
   )
-  (label "USR_LED_4" (at 109.22 130.81 180) (fields_autoplaced)
+  (label "USR_LED_2" (at 109.22 128.27 180) (fields_autoplaced)
     (effects (font (size 1.27 1.27)) (justify right bottom))
   )
@@
     (effects (font (size 1 1)) (justify right bottom))
   )
-  (label "USR_LED_1" (at 109.22 123.19 180) (fields_autoplaced)
-    (effects (font (size 1.27 1.27)) (justify right bottom))
-  )
   (label "SYS_JTMS-SWCLK" (at 88.9 73.66 270) (fields_autoplaced)
     (effects (font (size 1 1)) (justify right bottom))
@@
     (effects (font (size 1.27 1.27)) (justify left bottom))
   )
+  (label "USR_LED_4" (at 109.22 123.19 180) (fields_autoplaced)
+    (effects (font (size 1.27 1.27)) (justify right bottom))
+  )
+  (label "USR_LED_1" (at 109.22 130.81 180) (fields_autoplaced)
+    (effects (font (size 1.27 1.27)) (justify right bottom))
+  )
   (label "SYS_JTMS-SWDIO" (at 83.82 232.41 0) (fields_autoplaced)

Commit message: pcb update
Connections:
- net FDC_2: now also IC101.23 (PA7); no longer IC101.21 (PA5)
- net FDC_3: now also IC101.24 (PC4); no longer IC101.22 (PA6)
- net FDC_4: now also IC101.21 (PA5); no longer IC101.23 (PA7)
- net FDC_5: now also IC101.22 (PA6); no longer IC101.24 (PC4)
- net FDC_6: now also IC101.27 (PB1); no longer IC101.26 (PB0)
- net FDC_7: now also IC101.26 (PB0); no longer IC101.25 (PC5)
- net FDC_8: now also IC101.25 (PC5); no longer IC101.27 (PB1)
Changed lines of the file:
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@@
+    (effects (font (size 1.27 1.27)) (justify left bottom))
+  )
+  (label "FDC_1" (at 58.42 184.15 90) (fields_autoplaced)
     (effects (font (size 1.27 1.27)) (justify left bottom))
   )
@@
     (effects (font (size 1.27 1.27)) (justify left bottom))
   )
-  (label "FDC_5" (at 68.58 184.15 90) (fields_autoplaced)
-    (effects (font (size 1.27 1.27)) (justify left bottom))
-  )
   (label "USR_LED_3" (at 109.22 125.73 180) (fields_autoplaced)
     (effects (font (size 1.27 1.27)) (justify right bottom))
@@
     (effects (font (size 1.27 1.27)) (justify right bottom))
   )
-  (label "FDC_2" (at 60.96 184.15 90) (fields_autoplaced)
+  (label "FDC_3" (at 68.58 184.15 90) (fields_autoplaced)
     (effects (font (size 1.27 1.27)) (justify left bottom))
   )
@@
     (effects (font (size 1.27 1.27)) (justify right bottom))
   )
-  (label "FDC_8" (at 76.2 184.15 90) (fields_autoplaced)
-    (effects (font (size 1.27 1.27)) (justify left bottom))
-  )
   (label "FDC_3" (at 191.77 233.68 0) (fields_autoplaced)
     (effects (font (size 1.27 1.27)) (justify left bottom))
@@
     (effects (font (size 1.27 1.27)) (justify right bottom))
   )
-  (label "FDC_6" (at 73.66 184.15 90) (fields_autoplaced)
-    (effects (font (size 1.27 1.27)) (justify left bottom))
-  )
-  (label "FDC_1" (at 58.42 184.15 90) (fields_autoplaced)
+  (label "FDC_6" (at 76.2 184.15 90) (fields_autoplaced)
     (effects (font (size 1.27 1.27)) (justify left bottom))
   )
   (label "SYS_JTMS-SWDIO" (at 114.3 118.11 180) (fields_autoplaced)
     (effects (font (size 1 1)) (justify right bottom))
+  )
+  (label "FDC_2" (at 66.04 184.15 90) (fields_autoplaced)
+    (effects (font (size 1.27 1.27)) (justify left bottom))
   )
   (label "SYS_JTMS-SWCLK" (at 88.9 73.66 270) (fields_autoplaced)
@@
   (label "SYS_JTDO-SWO" (at 73.66 73.66 270) (fields_autoplaced)
     (effects (font (size 1 1)) (justify right bottom))
-  )
-  (label "FDC_7" (at 71.12 184.15 90) (fields_autoplaced)
-    (effects (font (size 1.27 1.27)) (justify left bottom))
   )
   (label "USR_LED_4" (at 109.22 123.19 180) (fields_autoplaced)
@@
     (effects (font (size 1.27 1.27)) (justify left bottom))
   )
+  (label "FDC_4" (at 60.96 184.15 90) (fields_autoplaced)
+    (effects (font (size 1.27 1.27)) (justify left bottom))
+  )
+  (label "FDC_8" (at 71.12 184.15 90) (fields_autoplaced)
+    (effects (font (size 1.27 1.27)) (justify left bottom))
+  )
   (label "FDC_4" (at 191.77 262.89 0) (fields_autoplaced)
     (effects (font (size 1.27 1.27)) (justify left bottom))
@@
     (effects (font (size 1 1)) (justify right bottom))
   )
-  (label "FDC_7" (at 243.84 236.22 0) (fields_autoplaced)
+  (label "FDC_7" (at 73.66 184.15 90) (fields_autoplaced)
     (effects (font (size 1.27 1.27)) (justify left bottom))
   )
-  (label "FDC_3" (at 63.5 184.15 90) (fields_autoplaced)
-    (effects (font (size 1.27 1.27)) (justify left bottom))
-  )
-  (label "FDC_4" (at 66.04 184.15 90) (fields_autoplaced)
+  (label "FDC_7" (at 243.84 236.22 0) (fields_autoplaced)
     (effects (font (size 1.27 1.27)) (justify left bottom))
   )
@@
     (effects (font (size 1 1)) (justify left bottom))
   )
+  (label "FDC_5" (at 63.5 184.15 90) (fields_autoplaced)
+    (effects (font (size 1.27 1.27)) (justify left bottom))
+  )
   (global_label "11.7V" (shape input) (at 227.33 129.54 180) (fields_autoplaced)

Commit message: update
Connections:
- net GPIO_CSN1: now also IC101.37 (PC6); no longer IC101.39 (PC8)
- net GPIO_CSN3: now also IC101.39 (PC8); no longer IC101.37 (PC6)
Changed lines of the file:
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@@
+    )
+  )
+  (global_label "GPIO_CSN3" (shape input) (at 96.52 135.89 0) (fields_autoplaced)
+    (effects (font (size 1.27 1.27)) (justify left))
+    (property "Intersheetrefs" "${INTERSHEET_REFS}" (at 109.8882 135.89 0)
+      (effects (font (size 1.27 1.27)) (justify left) hide)
     )
   )
@@
     )
   )
+  (global_label "GPIO_CSN1" (shape input) (at 96.52 140.97 0) (fields_autoplaced)
+    (effects (font (size 1.27 1.27)) (justify left))
+    (property "Intersheetrefs" "${INTERSHEET_REFS}" (at 109.8882 140.97 0)
+      (effects (font (size 1.27 1.27)) (justify left) hide)
+    )
+  )
   (global_label "GND7" (shape input) (at 266.7 241.3 0) (fields_autoplaced)
     (effects (font (size 1.27 1.27)) (justify left))
@@
     )
   )
-  (global_label "GPIO_CSN1" (shape input) (at 96.52 135.89 0) (fields_autoplaced)
-    (effects (font (size 1.27 1.27)) (justify left))
-    (property "Intersheetrefs" "${INTERSHEET_REFS}" (at 109.8882 135.89 0)
-      (effects (font (size 1.27 1.27)) (justify left) hide)
-    )
-  )
   (global_label "UART4_RX" (shape input) (at 96.52 250.19 180) (fields_autoplaced)
     (effects (font (size 1.27 1.27)) (justify right))
@@
       (effects (font (size 1.27 1.27)) (justify left) hide)
     )
-  )
-  (global_label "GPIO_CSN3" (shape input) (at 96.52 140.97 0) (fields_autoplaced)
-    (effects (font (size 1.27 1.27)) (justify left))
-    (property "Intersheetrefs" "${INTERSHEET_REFS}" (at 109.8882 140.97 0)
-      (effects (font (size 1.27 1.27)) (justify left) hide)
-    )
