File: Kicad/Eve/reg4.kicad_sch (KiCad schematic)
At the start: 11 parts, among them J8 Conn_01x03, J9 Conn_01x03

Commit message: updtated Kicad ver 7.11.23
Parts:
- removed C35: 220uF, Capacitor_SMD:CP_Elec_10x10.5, symbol Device:C_Polarized_Small
- removed C36: 10n, Capacitor_SMD:C_0603_1608Metric_Pad1.08x0.95mm_HandSolder, symbol Device:C_Small
- removed C37: 470uF, Capacitor_SMD:CP_Elec_10x10.5, symbol Device:C_Polarized_Small
- removed CR4: DST10100S, libs:DST10100S, symbol 2023-03-19_11-33-54:DST10100S
- removed J8, J9: Conn_01x03, symbol Connector_Generic:Conn_01x03
- removed L4: 22uH, Inductor_SMD:L_Wuerth_WE-PD-Typ-LS_Handsoldering, symbol Device:L_Small
- removed R17: 2.7k, Resistor_SMD:R_0603_1608Metric_Pad0.98x0.95mm_HandSolder, symbol Device:R_Small
- removed U7: ~, libs:LT1076CR-PBF, symbol custom:LT1076
- added C6: 220uF, Capacitor_SMD:CP_Elec_10x10.5, symbol Device:C_Polarized_Small
- added C7: 10n, Capacitor_SMD:C_0603_1608Metric_Pad1.08x0.95mm_HandSolder, symbol Device:C_Small
- added C8: 470uF, Capacitor_SMD:CP_Elec_10x10.5, symbol Device:C_Polarized_Small
- added CR1: DST10100S, TO277B_LTF, symbol 2023-03-19_11-33-54:DST10100S
- added D4: LED, LED_SMD:LED_0603_1608Metric_Pad1.05x0.95mm_HandSolder, symbol Device:LED
- added L1: 22uH, Inductor_SMD:L_Wuerth_WE-PD-Typ-LS_Handsoldering, symbol Device:L_Small
- added R5: 1k, Resistor_SMD:R_0603_1608Metric_Pad0.98x0.95mm_HandSolder, symbol Device:R_Small
- added R8: 2.7k, Resistor_SMD:R_0603_1608Metric_Pad0.98x0.95mm_HandSolder, symbol Device:R_Small
- added U1: ~, symbol custom:LT1076
- R18: value 23k -> 24k
Connections:
- net GND: now also C6.2, C7.2, C8.2, CR1.1, CR1.2, D4.1 (K), U1.4 (GND)
- net Vsw: now also CR1.3, L1.1, U1.2 (Vsw)
- net at R18.2, R19.1: now also U1.5 (FB)
- net 7.4V renamed 7.5V
- net 7.5V: now also C8.1, L1.2, R5.1
- new net: R8.1, U1.6 (Vc)
- new net: C7.1, R8.2
- new net: D4.2 (A), R5.2
- new net 24V: C6.1, U1.1 (Vin), U1.7 (Shutdown)
Other:
- moved on the sheet: R19

Commit message: added Kicad libraries to git + sch changes 11/11/23
Changed lines of the file:
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@@
   (junction (at 165.1 118.11) (diameter 0) (color 0 0 0 0)
-  )
-  (junction (at 165.1 85.09) (diameter 0) (color 0 0 0 0)
   )
   (junction (at 152.4 110.49) (diameter 0) (color 0 0 0 0)
@@
     (stroke (width 0) (type default))
   )
-  (wire (pts (xy 165.1 85.09) (xy 176.53 85.09))
-    (stroke (width 0) (type default))
-  )
   (wire (pts (xy 130.81 109.22) (xy 130.81 116.84))
     (stroke (width 0) (type default))
@@
     (effects (font (size 1.27 1.27)) (justify left bottom))
   )
-  (label "Vout" (at 166.37 85.09 0) (fields_autoplaced)
-    (effects (font (size 1.27 1.27)) (justify left bottom))
-  )
   (label "Vsw" (at 144.78 87.63 180) (fields_autoplaced)
-    (effects (font (size 1.27 1.27)) (justify right bottom))
-  )
-  (label "Vin" (at 110.49 88.9 0) (fields_autoplaced)
-    (effects (font (size 1.27 1.27)) (justify left bottom))
-  )
-  (label "7.5V" (at 176.53 85.09 0) (fields_autoplaced)
-    (effects (font (size 1.27 1.27)) (justify left bottom))
-  )
-  (label "7.5V" (at 226.06 81.28 270) (fields_autoplaced)
     (effects (font (size 1.27 1.27)) (justify right bottom))
   )
@@
     (effects (font (size 1.27 1.27)) (justify left))
   )
-  (hierarchical_label "7.5V" (shape input) (at 172.72 85.09 270) (fields_autoplaced)
-    (effects (font (size 1.27 1.27)) (justify right))
+  (hierarchical_label "7.5V" (shape input) (at 165.1 85.09 0) (fields_autoplaced)
+    (effects (font (size 1.27 1.27)) (justify left))
+  )
+  (hierarchical_label "7.5V" (shape input) (at 226.06 81.28 90) (fields_autoplaced)
+    (effects (font (size 1.27 1.27)) (justify left))
   )
   (symbol (lib_id "power:GND") (at 165.1 133.35 0) (unit 1)

Commit message: empreinte 13/11
Parts:
- C6: value 220uF -> 220u
- C8: value 470uF -> 470u
- CR1: footprint TO277B_LTF -> libs:DST10100S
- L1: footprint Inductor_SMD:L_Wuerth_WE-PD-Typ-LS_Handsoldering -> (none)
- U1: footprint (none) -> libs:LT1076CR-PBF
Changed lines of the file:
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@@
       (effects (font (size 1.27 1.27)) (justify left))
     )
-    (property "Value" "470uF" (at 157.48 95.25 0)
+    (property "Value" "470u" (at 157.48 95.25 0)
       (effects (font (size 1.27 1.27)) (justify left))
     )
@@
       (effects (font (size 1.27 1.27)))
     )
-    (property "Footprint" "Inductor_SMD:L_Wuerth_WE-PD-Typ-LS_Handsoldering" (at 151.13 85.09 0)
+    (property "Footprint" "" (at 151.13 85.09 0)
       (effects (font (size 1.27 1.27)) hide)
     )
@@
       (effects (font (size 1.27 1.27)))
     )
-    (property "Footprint" "" (at 125.73 92.71 0)
+    (property "Footprint" "libs:LT1076CR-PBF" (at 125.73 92.71 0)
       (effects (font (size 1.27 1.27)) hide)
     )
@@
       (effects (font (size 1.524 1.524)) (justify right))
     )
-    (property "Footprint" "TO277B_LTF" (at 141.224 97.79 0)
+    (property "Footprint" "libs:DST10100S" (at 141.224 97.79 0)
       (effects (font (size 1.524 1.524)) hide)
     )
@@
       (effects (font (size 1.27 1.27)) (justify left))
     )
-    (property "Value" "220uF" (at 106.68 97.7011 0)
-      (effects (font (size 1.27 1.27)) (justify left))
-    )
+    (property "Value" "220u" (at 106.68 97.7011 0)
+      (effects (font (size 1.27 1.27)) (justify left))
+    )

Commit message: pulled main and started routing
Parts:
- L1: footprint (none) -> Eagle_WE-PD (rev23a):WE-PD_1210
Changed lines of the file:
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@@
       (effects (font (size 1.27 1.27)))
     )
-    (property "Footprint" "" (at 151.13 85.09 0)
+    (property "Footprint" "Eagle_WE-PD (rev23a):WE-PD_1210" (at 151.13 85.09 0)
       (effects (font (size 1.27 1.27)) hide)
     )

Commit message: EVE 2.0 WIP
Parts:
- R5: value 1k -> 375
Changed lines of the file:
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@@
   (symbol (lib_id "Device:R_Small") (at 226.06 87.63 0) (unit 1)
     (in_bom yes) (on_board yes) (dnp no) (fields_autoplaced)
-    (property "Reference" "R5" (at 228.6 86.995 0)
+    (property "Reference" "R5" (at 228.6 86.36 0)
       (effects (font (size 1.27 1.27)) (justify left))
     )
-    (property "Value" "1k" (at 228.6 89.535 0)
+    (property "Value" "375" (at 228.6 88.9 0)
       (effects (font (size 1.27 1.27)) (justify left))
     )

Commit message: update pcb
Parts:
- C?: renamed from C7; footprint Capacitor_SMD:C_0603_1608Metric_Pad1.08x0.95mm_HandSolder -> Capacitor_SMD:C_0402_1005Metric
- CR?: renamed from CR1; footprint libs:DST10100S -> DST10100S:DST10100S
- D?: renamed from D4; footprint LED_SMD:LED_0603_1608Metric_Pad1.05x0.95mm_HandSolder -> LED_SMD:LED_0603_1608Metric
- L?: renamed from L1; footprint Eagle_WE-PD (rev23a):WE-PD_1210 -> Inductor_SMD:L_12x12mm_H8mm
- R802: renamed from R18; footprint Resistor_SMD:R_0603_1608Metric_Pad0.98x0.95mm_HandSolder -> Resistor_SMD:R_0402_1005Metric
- R803: renamed from R19; footprint Resistor_SMD:R_0603_1608Metric_Pad0.98x0.95mm_HandSolder -> Resistor_SMD:R_0402_1005Metric
- R?: renamed from R8; footprint Resistor_SMD:R_0603_1608Metric_Pad0.98x0.95mm_HandSolder -> Resistor_SMD:R_0402_1005Metric
- R?: renamed from R5; footprint Resistor_SMD:R_0603_1608Metric_Pad0.98x0.95mm_HandSolder -> Resistor_SMD:R_0402_1005Metric
- U?: renamed from U1; value ~ -> LT1076CR-PBF; footprint libs:LT1076CR-PBF -> LT1076CR:LT1076CR-PBF
- renumbered C8 to C?, C6 to C?

Commit message: update 18/12
Parts:
- R?: value 375 -> 1.5k
Changed lines of the file:
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@@
   (symbol (lib_id "Device:R_Small") (at 226.06 87.63 0) (unit 1)
     (in_bom yes) (on_board yes) (dnp no) (fields_autoplaced)
-    (property "Reference" "R?" (at 228.6 86.36 0)
+    (property "Reference" "R?" (at 228.6 86.995 0)
       (effects (font (size 1.27 1.27)) (justify left))
     )
-    (property "Value" "375" (at 228.6 88.9 0)
+    (property "Value" "1.5k" (at 228.6 89.535 0)
       (effects (font (size 1.27 1.27)) (justify left))
     )
