File: Kicad/Eve/reg4.kicad_sch (KiCad schematic)
At the start: 11 parts

Commit message: update PCB
Parts:
- C?: value 470u -> 47u; footprint Capacitor_SMD:CP_Elec_10x10.5 -> Capacitor_SMD:CP_Elec_6.3x5.4; MFR 865060457009 -> 865060543005
- C?: value 220u -> 100u; footprint Capacitor_SMD:CP_Elec_10x10.5 -> Capacitor_SMD:CP_Elec_6.3x7.7; MFR 865060657012 -> 865060445005; Vmax 50V -> 25V
- L?: footprint Inductor_SMD:L_12x12mm_H8mm -> Inductor_SMD:L_Changjiang_FNR8065S
Changed lines of the file:
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@@
       (effects (font (size 1.27 1.27)) (justify left))
     )
-    (property "Value" "470u" (at 157.48 95.25 0)
-      (effects (font (size 1.27 1.27)) (justify left))
-    )
-    (property "Footprint" "Capacitor_SMD:CP_Elec_10x10.5" (at 154.94 93.98 0)
+    (property "Value" "47u" (at 157.48 95.25 0)
+      (effects (font (size 1.27 1.27)) (justify left))
+    )
+    (property "Footprint" "Capacitor_SMD:CP_Elec_6.3x5.4" (at 154.94 93.98 0)
       (effects (font (size 1.27 1.27)) hide)
     )
@@
       (effects (font (size 1.27 1.27)) hide)
     )
-    (property "MFR" "865060457009" (at 154.94 93.98 0)
+    (property "MFR" "865060543005" (at 154.94 93.98 0)
       (effects (font (size 1.27 1.27)) hide)
     )
@@
       (effects (font (size 1.27 1.27)))
     )
-    (property "Footprint" "Inductor_SMD:L_12x12mm_H8mm" (at 151.13 85.09 0)
+    (property "Footprint" "Inductor_SMD:L_Changjiang_FNR8065S" (at 151.13 85.09 0)
       (effects (font (size 1.27 1.27)) hide)
     )
@@
       (effects (font (size 1.27 1.27)) (justify left))
     )
-    (property "Value" "220u" (at 106.68 97.7011 0)
-      (effects (font (size 1.27 1.27)) (justify left))
-    )
-    (property "Footprint" "Capacitor_SMD:CP_Elec_10x10.5" (at 114.3 93.98 0)
+    (property "Value" "100u" (at 106.68 97.7011 0)
+      (effects (font (size 1.27 1.27)) (justify left))
+    )
+    (property "Footprint" "Capacitor_SMD:CP_Elec_6.3x7.7" (at 114.3 93.98 0)
       (effects (font (size 1.27 1.27)) hide)
     )
@@
       (effects (font (size 1.27 1.27)) hide)
     )
-    (property "MFR" "865060657012" (at 114.3 93.98 0)
-      (effects (font (size 1.27 1.27)) hide)
-    )
-    (property "Vmax" "50V" (at 114.3 93.98 0)
-      (effects (font (size 1.27 1.27)) hide)
-    )
+    (property "MFR" "865060445005" (at 114.3 93.98 0)
+      (effects (font (size 1.27 1.27)) hide)
+    )
+    (property "Vmax" "25V" (at 114.3 93.98 0)
+      (effects (font (size 1.27 1.27)) hide)
+    )
