File: Kicad/Eve/Robourt.kicad_pcb (KiCad board)
At the start: 4 copper layers, 85 x 70 mm, 172 parts, among them IC101 STM32U535RET6, J1 Conn_02x08_Odd_Even, J101 Conn_ST_STDC14, J102 Conn_01x02, J103 Conn_01x02, J108 Conn_01x03, J109 Conn_01x03, J110 Conn_01x02, J115 Conn_02x20_Odd_Even, J201 Conn_01x04, J301 Conn_01x04, J401 Conn_01x04, Q101 NMOS, Q201 SQJ504EP-T1_GE3, Q202 SQJ504EP-T1_GE3, Q203 SQJ504EP-T1_GE3, Q204 SQJ504EP-T1_GE3, Q301 SQJ504EP-T1_GE3, Q302 SQJ504EP-T1_GE3, Q303 SQJ504EP-T1_GE3, Q304 SQJ504EP-T1_GE3, Q401 SQJ504EP-T1_GE3, Q402 SQJ504EP-T1_GE3, Q403 SQJ504EP-T1_GE3, Q404 SQJ504EP-T1_GE3, SW101 SW_Push, SW102 SW_Push, SW103 SW_Push, SW104 SW_Push, U201 TMC2590-TA, U301 TMC2590-TA, U401 TMC2590-TA, U501 BU33SD5WG-TR, U601 LT1076CR-PBF, U701 LT1076CR-PBF, U801 LT1076CR-PBF, Y101 Crystal

Commit message: lib working for all + PCB progress
Parts:
- C205: value 150u -> locked
- C301, C302, C303, C306, C307, C308, C309, C401, C402, C403, C406, C407, C408, C409, R301, R302, R303, R304, R401, R402, R403, R404, U301, U401: moved to B.Cu
- J1: footprint Connector_PinSocket_2.54mm:PinSocket_2x08_P2.54mm_Vertical_SMD -> Connector_PinHeader_2.00mm:PinHeader_2x08_P2.00mm_Vertical_SMD
- moved R102 210.8 mm to (97.8, -65.5)
- moved R104 210.8 mm to (97.8, -61.6)
- moved C104 210.8 mm to (103.7, -83.0)
- moved SW102 210.8 mm to (99.3, -79.4)
- moved Q301 200.8 mm to (66.2, 45.8)
- moved Q401 198.9 mm to (43.5, 45.8)
- moved C405 197.3 mm to (35.0, 26.9), turned to -90 degrees
- moved Q402 195.7 mm to (43.4, 22.6), turned to 180 degrees
- moved C113 193.0 mm to (-52.6, 80.2)
- moved C114 193.0 mm to (-52.0, 94.5)
- moved C115 193.0 mm to (-8.62, 81.6)
- moved C118 193.0 mm to (-19.9, 99.9)
- moved C119 193.0 mm to (-55.6, 111.3)
- moved R116 193.0 mm to (-52.6, 83.0)
- moved R117 193.0 mm to (-52.1, 98.1)
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Connections:
- Q202 pad 3: Net-(Q202-S2) -> /driver_stepper/S
- Q202 pad 4: /driver_stepper/B1 -> /driver_stepper/HB1
- Q202 pad 6: /driver_stepper/HB1 -> /driver_stepper/B1
- Q204 pad 1: Net-(Q202-S2) -> /driver_stepper/S
- Q302 pad 3: Net-(Q302-S2) -> /driver_stepper1/S
- Q302 pad 4: /driver_stepper1/B1 -> /driver_stepper1/HB1
- Q302 pad 6: /driver_stepper1/HB1 -> /driver_stepper1/B1
- Q304 pad 1: Net-(Q302-S2) -> /driver_stepper1/S
- Q402 pad 3: Net-(Q402-S2) -> /driver_stepper2/S
- Q402 pad 4: /driver_stepper2/B1 -> /driver_stepper2/HB1
- Q402 pad 6: /driver_stepper2/HB1 -> /driver_stepper2/B1
- Q404 pad 1: Net-(Q402-S2) -> /driver_stepper2/S
Routing:
- net GND: track 31.9 -> 95.6 mm, vias 9 -> 27
- net /driver_stepper2/LB1: track 0.00 -> 35.6 mm, vias 0 -> 2
- net /driver_stepper2/B2: track 0.00 -> 35.0 mm, vias 0 -> 2
- net /driver_stepper1/LB1: track 0.00 -> 34.3 mm, vias 0 -> 2
- net /driver_stepper1/B2: track 0.00 -> 34.2 mm, vias 0 -> 2
- net /driver_stepper2/B1: track 0.00 -> 33.2 mm, vias 0 -> 1
- net /driver_stepper2/LB2: track 0.00 -> 32.2 mm, vias 0 -> 2
- net /driver_stepper1/LB2: track 0.00 -> 31.3 mm, vias 0 -> 2
- net /driver_stepper2/HB2: track 0.00 -> 27.4 mm, vias 0 -> 2
- net /driver_stepper1/HB2: track 0.00 -> 26.8 mm, vias 0 -> 2
- net 24V: track 11.9 -> 35.6 mm, vias 10 -> 30
- net /driver_stepper2/SRB: track 0.00 -> 22.4 mm, vias 0 -> 2
- net /driver_stepper1/SRB: track 0.00 -> 22.1 mm, vias 0 -> 2
- net /driver_stepper2/A2: track 0.00 -> 20.9 mm, vias 0 -> 2
- net /driver_stepper1/A2: track 0.00 -> 20.7 mm, vias 0 -> 2
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
Commit message: update 17/12
Parts:
- C101, C102, C105, C106, C107, C108, C116, C117, R124, Y101: moved to B.Cu
- moved C119 215.7 mm to (158.6, 85.6)
- moved R130 215.7 mm to (158.5, 86.8)
- moved R126 215.7 mm to (158.4, 88.0)
- moved C120 206.9 mm to (158.0, 90.3)
- moved R127 206.9 mm to (158.1, 93.0)
- moved R131 206.9 mm to (157.9, 91.6)
- moved C113 202.0 mm to (149.3, 84.6)
- moved R116 202.0 mm to (149.4, 87.4)
- moved R121 202.0 mm to (149.5, 86.1)
- moved C114 201.5 mm to (149.5, 90.3)
- moved R117 201.5 mm to (149.4, 93.9)
- moved R122 201.5 mm to (149.5, 91.8)
- moved R128 186.7 mm to (158.0, 98.2)
- moved C121 186.7 mm to (157.6, 96.2)
- moved R132 186.7 mm to (158.1, 100.2)
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Connections:
- C101 pad 2: GND -> GND1
- C102 pad 2: GND -> GND1
- C103 pad 2: GND -> GND1
- C104 pad 2: GND -> GND1
- C105 pad 2: GND -> GND1
- C106 pad 2: GND -> GND1
- C107 pad 2: GND -> GND1
- C108 pad 2: GND -> GND1
- C109 pad 2: GND -> GND1
- C110 pad 2: GND -> GND1
- C111 pad 2: GND -> GND1
- C112 pad 2: GND -> GND1
- C113 pad 2: GND -> GND1
- C114 pad 2: GND -> GND1
- C115 pad 2: GND -> GND1
- C116 pad 2: GND -> GND1
- C117 pad 2: GND -> GND1
- C118 pad 2: GND -> GND1
- C119 pad 2: GND -> GND1
- C120 pad 2: GND -> GND1
- C121 pad 2: GND -> GND1
- C201 pad 2: GND -> GND1
- C202 pad 2: GND -> GND1
- C203 pad 2: GND -> GND1
- C204 pad 2: GND -> GND1
- C205 pad 2: GND -> GND1
- C207 pad 2: GND -> GND1
- C208 pad 2: GND -> GND1
- C209 pad 2: GND -> GND1
- C301 pad 2: GND -> GND1
- C302 pad 2: GND -> GND1
- C303 pad 2: GND -> GND1
- C304 pad 2: GND -> GND1
- C305 pad 2: GND -> GND1
- C307 pad 2: GND -> GND1
- C308 pad 2: GND -> GND1
- C309 pad 2: GND -> GND1
- C401 pad 2: GND -> GND1
- C402 pad 2: GND -> GND1
- C403 pad 2: GND -> GND1
- C404 pad 2: GND -> GND1
- C405 pad 2: GND -> GND1
- C407 pad 2: GND -> GND1
- C408 pad 2: GND -> GND1
- C409 pad 2: GND -> GND1
- C501 pad 2: GND -> GND1
- C502 pad 2: GND -> GND1
- C601 pad 2: GND -> GND1
- C602 pad 2: GND -> GND1
- C603 pad 2: GND -> GND1
- C701 pad 2: GND -> GND1
- C702 pad 2: GND -> GND1
- C703 pad 2: GND -> GND1
- C801 pad 2: GND -> GND1
- C802 pad 2: GND -> GND1
- C803 pad 2: GND -> GND1
- CR601 pad 1: GND -> GND1
- CR601 pad 2: GND -> GND1
- CR701 pad 1: GND -> GND1
- CR701 pad 2: GND -> GND1
- CR801 pad 1: GND -> GND1
- CR801 pad 2: GND -> GND1
- D105 pad 1: GND -> GND1
- D501 pad 1: GND -> GND1
- D601 pad 1: GND -> GND1
- D701 pad 1: GND -> GND1
- D801 pad 1: GND -> GND1
- H101 pad 1: GND -> GND1
- H102 pad 1: GND -> GND1
- H103 pad 1: GND -> GND1
- H104 pad 1: GND -> GND1
- IC101 pad 12: GND -> GND1
- IC101 pad 18: GND -> GND1
- IC101 pad 31: GND -> GND1
- IC101 pad 47: GND -> GND1
- IC101 pad 60: GND -> GND1
- IC101 pad 63: GND -> GND1
- J1 pad 1: unconnected-(J1-Pin_1-Pad1) -> FDC1
- J1 pad 10: unconnected-(J1-Pin_10-Pad10) -> GND1
- J1 pad 11: unconnected-(J1-Pin_11-Pad11) -> FDC6
- J1 pad 12: unconnected-(J1-Pin_12-Pad12) -> GND1
- J1 pad 13: unconnected-(J1-Pin_13-Pad13) -> FDC7
- J1 pad 14: unconnected-(J1-Pin_14-Pad14) -> GND1
- J1 pad 15: unconnected-(J1-Pin_15-Pad15) -> FDC8
- J1 pad 16: unconnected-(J1-Pin_16-Pad16) -> GND1
- J1 pad 2: unconnected-(J1-Pin_2-Pad2) -> GND1
- J1 pad 3: unconnected-(J1-Pin_3-Pad3) -> FDC2
- J1 pad 4: unconnected-(J1-Pin_4-Pad4) -> GND1
- J1 pad 5: unconnected-(J1-Pin_5-Pad5) -> FDC3
- J1 pad 6: unconnected-(J1-Pin_6-Pad6) -> GND1
- J1 pad 7: unconnected-(J1-Pin_7-Pad7) -> FDC4
- J1 pad 8: unconnected-(J1-Pin_8-Pad8) -> GND1
- J1 pad 9: unconnected-(J1-Pin_9-Pad9) -> FDC5
- J101 pad 11: GND -> GND1
- J101 pad 5: GND -> GND1
- J101 pad 7: GND -> GND1
- J108 pad 3: GND -> GND1
- J109 pad 3: GND -> GND1
- J110 pad 1: GND -> GND1
- J115 pad 14: GND -> GND1
- J115 pad 20: GND -> GND1
- J115 pad 25: GND -> GND1
- J115 pad 30: GND -> GND1
- J115 pad 34: GND -> GND1
- J115 pad 39: GND -> GND1
- J115 pad 6: GND -> GND1
- J115 pad 9: GND -> GND1
- Q101 pad 3: GND -> GND1
- R105 pad 2: GND -> GND1
- R106 pad 2: GND -> GND1
- R108 pad 2: GND -> GND1
- R109 pad 2: GND -> GND1
- R114 pad 2: GND -> GND1
- R120 pad 2: unconnected-(R120-Pad2) -> FDC1
- R121 pad 2: unconnected-(R121-Pad2) -> FDC2
- R122 pad 2: unconnected-(R122-Pad2) -> FDC3
- R123 pad 2: unconnected-(R123-Pad2) -> FDC4
- R129 pad 2: unconnected-(R129-Pad2) -> FDC5
- R130 pad 2: unconnected-(R130-Pad2) -> FDC6
- R131 pad 2: unconnected-(R131-Pad2) -> FDC7
- R132 pad 2: unconnected-(R132-Pad2) -> FDC8
- R201 pad 2: GND -> GND1
- R202 pad 2: GND -> GND1
- R301 pad 2: GND -> GND1
- R302 pad 2: GND -> GND1
- R401 pad 2: GND -> GND1
- R402 pad 2: GND -> GND1
- R603 pad 2: GND -> GND1
- R703 pad 2: GND -> GND1
- R803 pad 2: GND -> GND1
- SW101 pad 2: GND -> GND1
- SW102 pad 2: GND -> GND1
- SW103 pad 2: GND -> GND1
- SW104 pad 2: GND -> GND1
- U201 pad 1: GND -> GND1
- U201 pad 13: GND -> GND1
- U201 pad 15: GND -> GND1
- U201 pad 28: GND -> GND1
- U201 pad 32: GND -> GND1
- U201 pad 33: GND -> GND1
- U301 pad 1: GND -> GND1
- U301 pad 13: GND -> GND1
- U301 pad 15: GND -> GND1
- U301 pad 28: GND -> GND1
- U301 pad 32: GND -> GND1
- U301 pad 33: GND -> GND1
- U401 pad 1: GND -> GND1
- U401 pad 13: GND -> GND1
- U401 pad 15: GND -> GND1
- U401 pad 28: GND -> GND1
- U401 pad 32: GND -> GND1
- U401 pad 33: GND -> GND1
- U501 pad 2: GND -> GND1
- U601 pad 4: GND -> GND1
- U701 pad 4: GND -> GND1
- U801 pad 4: GND -> GND1
- Y101 pad 2: GND -> GND1
- Y101 pad 4: GND -> GND1
Routing:
- net GND1: track 0.00 -> 106.0 mm, vias 0 -> 27
- net GND: track 95.6 -> 0.00 mm, vias 27 -> 0
- net /NRST: track 4.24 -> 0.00 mm
- net /USR_BTN_3: track 4.08 -> 0.00 mm
- net /USR_LED_1: track 3.61 -> 0.00 mm
- net /USR_LED_4: track 3.58 -> 0.00 mm
- net /USR_LED_2: track 3.16 -> 0.00 mm
- net /USR_LED_3: track 3.13 -> 0.00 mm
- net +3.3V: track 12.5 -> 15.3 mm
- net /Vcap: track 1.76 -> 0.00 mm
- net Net-(C117-Pad1): track 3.49 -> 5.09 mm
- net Net-(R103-Pad2): track 1.38 -> 0.00 mm
- net OSC_in: track 6.06 -> 4.79 mm
- net OSC_out: track 2.83 -> 1.71 mm
- added copper zone on B.Cu, net GND1
- added copper zone on F.Cu, net GND1
- added copper zone on In1.Cu, net GND1
- removed copper zone on B.Cu, net GND
- removed copper zone on F.Cu, net GND
- removed copper zone on In1.Cu, net GND

Commit message: update 18/12
Parts:
- C111: moved to B.Cu
- R119: value 1k -> 4k
- R704: value 680 -> 2k
- R804: value 375 -> 1.5k
- moved C111 175.0 mm to (96.5, 71.6)
- moved SW103 100.9 mm to (46.6, -19.5)
- moved R112 99.2 mm to (47.5, -13.6)
- moved C109 99.2 mm to (48.4, -16.6)
- moved SW101 98.4 mm to (49.6, -39.5)
- moved C103 98.4 mm to (44.6, -39.8)
- moved C110 98.4 mm to (33.5, -30.9)
- moved D101 98.4 mm to (27.4, -36.2)
- moved D102 98.4 mm to (27.4, -37.7)
- moved D103 98.4 mm to (27.4, -39.4)
- moved D104 98.4 mm to (27.4, -41.0)
- moved R101 98.4 mm to (45.6, -40.9)
- moved R103 98.4 mm to (46.1, -39.4)
- moved R106 98.4 mm to (25.2, -37.6)
- moved R109 98.4 mm to (25.2, -41.6)
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Routing:
- net /FDC_5: track 0.00 -> 51.8 mm, vias 0 -> 1
- net /FDC_4: track 0.00 -> 51.5 mm, vias 0 -> 1
- net +3.3V: track 15.3 -> 56.6 mm, vias 0 -> 1
- net /FDC_8: track 0.00 -> 33.0 mm, vias 0 -> 2
- net /FDC_6: track 0.00 -> 29.8 mm, vias 0 -> 2
- net /FDC_7: track 0.00 -> 28.9 mm, vias 0 -> 1
- net /FDC_3: track 0.00 -> 28.2 mm, vias 0 -> 1
- net /FDC_1: track 0.00 -> 28.1 mm, vias 0 -> 1
- net FDC1: track 0.00 -> 17.4 mm
- net FDC2: track 0.00 -> 15.4 mm
- net FDC3: track 0.00 -> 14.1 mm
- net FDC5: track 0.00 -> 11.7 mm
- net FDC6: track 0.00 -> 9.47 mm
- net FDC4: track 0.00 -> 9.27 mm
- net FDC7: track 0.00 -> 6.32 mm
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
Commit message: PCB tried some layout
Parts:
- C110, C803, CR801, L801, R111, R113: moved to B.Cu
- moved Q101 60.7 mm to (24.5, 69.9)
- moved R108 57.8 mm to (23.5, 72.3)
- moved R107 56.8 mm to (23.5, 67.4)
- moved J102 28.3 mm to (-10.2, 33.1)
- moved J103 27.6 mm to (-10.8, 41.2)
- moved C801 25.8 mm to (131.9, 31.3), turned to 90 degrees
- moved C501 22.8 mm to (191.2, 20.9)
- moved D501 22.7 mm to (196.0, 24.6)
- moved C502 22.7 mm to (197.1, 21.0)
- moved U501 22.7 mm to (194.5, 22.1)
- moved R501 22.7 mm to (197.0, 22.9)
- moved D801 20.0 mm to (133.4, 24.9), turned to 0 degrees
- moved R804 19.9 mm to (136.0, 25.1)
- moved L801 18.3 mm to (131.1, 30.4), turned to 90 degrees
- moved C803 12.1 mm to (143.5, 29.4), turned to -90 degrees
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Routing:
- net Net-(U801-FB): track 0.00 -> 8.92 mm
- net 7.5V: track 0.00 -> 8.19 mm, vias 0 -> 1
- net Net-(U801-Vc): track 0.00 -> 3.94 mm
- net Net-(R113-Pad2): track 0.00 -> 2.71 mm, vias 0 -> 1
- net /USR_BTN_3: track 0.00 -> 2.25 mm
- net Net-(C802-Pad1): track 0.00 -> 1.01 mm

Commit message: PCB cleaning
Parts:
- moved Q204 0.17 mm to (94.6, 22.7)
- moved Q202 0.17 mm to (88.8, 22.7)
- moved Q303 0.15 mm to (72.1, 45.8)
- moved R301 0.15 mm to (69.1, 42.7)
- moved R302 0.15 mm to (69.1, 25.6)
- moved C303 0.15 mm to (57.7, 26.9)
- moved C305 0.15 mm to (57.7, 26.9)
- moved R304 0.15 mm to (62.6, 26.0)
- moved U301 0.15 mm to (57.8, 40.4)
- moved C301 0.14 mm to (69.1, 23.1)
- moved C302 0.14 mm to (69.2, 45.2)
- moved C304 0.14 mm to (57.9, 40.4)
- moved C306 0.14 mm to (53.1, 37.5)
- moved C307 0.14 mm to (56.0, 35.7)
- moved C308 0.14 mm to (60.3, 45.3)
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Routing:
- net /driver_stepper1/B1: track 19.2 -> 26.6 mm
- net /driver_stepper2/B1: track 33.2 -> 26.7 mm
- net /driver_stepper2/HB1: track 18.2 -> 23.4 mm
- net /driver_stepper1/HB1: track 18.1 -> 23.2 mm
- net /driver_stepper/HB1: track 17.9 -> 23.0 mm
- net /driver_stepper/B1: track 32.9 -> 29.7 mm
- net /driver_stepper1/LB1: track 34.3 -> 35.1 mm
- net /driver_stepper1/LB2: track 31.3 -> 32.0 mm

Commit message: update 19/12
Parts:
- moved C501 0.95 mm to (191.8, 21.6)
Changed lines of the file:
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@@
   )
   (footprint "Capacitor_SMD:C_0402_1005Metric" (layer "F.Cu")
-    (at 191.225 20.85 -90)
+    (at 191.8 21.6 -90)
     (descr "Capacitor SMD 0402 (1005 Metric), square (rectangular) end terminal, IPC_7351 nominal, (Body size source: IPC-SM-782 page 76, https://www.pcb-3d.com/wordpress/wp-content/uploads/ipc-sm-782a_amendment_1_and_2.pdf), generated with kicad-footprint-generator")
     (tags "capacitor")
@@
   )
   (footprint "Resistor_SMD:R_0402_1005Metric" (layer "F.Cu")
-    (at 197.045 22.9 -90)
+    (at 197.06 22.9 -90)
     (descr "Resistor SMD 0402 (1005 Metric), square (rectangular) end terminal, IPC_7351 nominal, (Body size source: IPC-SM-782 page 72, https://www.pcb-3d.com/wordpress/wp-content/uploads/ipc-sm-782a_amendment_1_and_2.pdf), generated with kicad-footprint-generator")
     (tags "resistor")
