File: Kicad/Eve/Robourt.kicad_pcb (KiCad board)
At the start: 4 copper layers, 85 x 70 mm, 172 parts, among them IC101 STM32U535RET6, J1 Conn_02x08_Odd_Even, J101 Conn_ST_STDC14, J102 Conn_01x02, J103 Conn_01x02, J108 Conn_01x03, J109 Conn_01x03, J110 Conn_01x02, J115 Conn_02x20_Odd_Even, J201 Conn_01x04, J301 Conn_01x04, J401 Conn_01x04, Q101 NMOS, Q201 SQJ504EP-T1_GE3, Q202 SQJ504EP-T1_GE3, Q203 SQJ504EP-T1_GE3, Q204 SQJ504EP-T1_GE3, Q301 SQJ504EP-T1_GE3, Q302 SQJ504EP-T1_GE3, Q303 SQJ504EP-T1_GE3, Q304 SQJ504EP-T1_GE3, Q401 SQJ504EP-T1_GE3, Q402 SQJ504EP-T1_GE3, Q403 SQJ504EP-T1_GE3, Q404 SQJ504EP-T1_GE3, SW101 SW_Push, SW102 SW_Push, SW103 SW_Push, SW104 SW_Push, U201 TMC2590-TA, U301 TMC2590-TA, U401 TMC2590-TA, U501 BU33SD5WG-TR, U601 LT1076CR-PBF, U701 LT1076CR-PBF, U801 LT1076CR-PBF, Y101 Crystal

Commit message: update cha 19/12
Parts:
- C603, CR601, L601: moved to B.Cu
- moved C602 88.2 mm to (135.2, 24.5)
- moved R601 85.4 mm to (137.2, 24.5), turned to 180 degrees
- moved R603 80.8 mm to (137.2, 14.2)
- moved R602 77.3 mm to (135.2, 14.2), turned to 0 degrees
- moved U601 71.8 mm to (144.3, 19.3), turned to -90 degrees
- moved D601 68.5 mm to (150.0, 10.0), turned to -90 degrees
- moved R604 66.0 mm to (150.0, 12.5)
- moved CR601 63.5 mm to (136.6, 18.8), turned to 180 degrees
- moved L601 59.8 mm to (143.5, 7.02), turned to 0 degrees
- moved C601 53.9 mm to (143.6, 6.90), turned to 0 degrees
- moved C603 47.8 mm to (145.5, 19.2), turned to 180 degrees
- moved C801 8.68 mm to (125.0, 36.6)
- moved C803 7.91 mm to (137.6, 34.7)
- moved R802 7.76 mm to (132.2, 44.9)
- moved R803 7.76 mm to (132.2, 42.9)
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Routing:
- net GND1: track 107.4 -> 192.4 mm, vias 27 -> 33
- net 5.1V: track 0.00 -> 35.1 mm
- net 7.5V: track 8.19 -> 36.5 mm
- net /Régulateur 7.5V/Vsw: track 0.00 -> 21.1 mm, vias 0 -> 1
- net /Régulateur 5.1V/Vsw: track 0.00 -> 21.0 mm, vias 0 -> 1
- net Net-(U601-FB): track 0.00 -> 8.87 mm
- net Net-(U601-Vc): track 0.00 -> 4.55 mm
- net +3.3V: track 56.6 -> 59.1 mm
- net Net-(D801-A): track 0.00 -> 1.39 mm
- net Net-(D501-A): track 0.00 -> 1.34 mm
- net Net-(D601-A): track 0.00 -> 1.20 mm
- net Net-(C602-Pad1): track 0.00 -> 1.01 mm

Commit message: small PCB update
Parts:
- moved R111 143.8 mm to (151.8, 55.5)
- moved R113 143.8 mm to (150.2, 56.1)
- moved SW104 143.8 mm to (151.2, 56.0)
- moved C110 131.1 mm to (99.0, 87.7), turned to -90 degrees
- moved R604 119.9 mm to (43.3, 67.2), turned to 0 degrees
- moved D601 118.9 mm to (45.8, 67.2), turned to 180 degrees
- moved C603 116.6 mm to (36.8, 61.2), turned to 90 degrees
- moved U601 115.7 mm to (36.7, 61.8), turned to 180 degrees
- moved R601 109.9 mm to (31.6, 54.7), turned to 90 degrees
- moved C601 108.8 mm to (49.1, 60.9), turned to -90 degrees
- moved L601 108.0 mm to (49.0, 59.2), turned to -90 degrees
- moved C602 107.4 mm to (31.6, 52.7), turned to 90 degrees
- moved CR601 104.9 mm to (37.2, 52.3), turned to 90 degrees
- moved R603 103.7 mm to (41.8, 54.7), turned to -90 degrees
- moved R602 101.0 mm to (41.8, 52.7), turned to -90 degrees
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Routing:
- net GND1: track 192.4 -> 180.7 mm
- net 24V: track 35.4 -> 41.7 mm, vias 30 -> 33
- net /FDC_1: track 28.1 -> 31.8 mm
- net /USR_BTN_3: track 2.25 -> 0.00 mm
- net Net-(U601-FB): track 8.87 -> 11.1 mm, vias 0 -> 1
- net /Régulateur 5.1V/Vsw: track 21.0 -> 18.8 mm
- net 5.1V: track 35.1 -> 35.2 mm, vias 0 -> 1

Commit message: update PCB
Parts:
- removed C601, C701: 220u, Capacitor_SMD:CP_Elec_10x10.5
- added C604: 100u, Capacitor_SMD:CP_Elec_6.3x7.7, F.Cu at (43.1, 52.0)
- added C704: 100u, Capacitor_SMD:CP_Elec_6.3x7.7, F.Cu at (75.4, 52.0)
- C103, C104, C109, CR701, R101, R102, R103, R104, R110, R112: moved to B.Cu
- C603, C803: value 470u -> 47u; footprint Capacitor_SMD:CP_Elec_10x10.5 -> Capacitor_SMD:CP_Elec_6.3x5.4; moved to F.Cu
- C703: value 470u -> 47u; footprint Capacitor_SMD:CP_Elec_10x10.5 -> Capacitor_SMD:CP_Elec_6.3x5.4
- C801: value 220u -> 100u; footprint Capacitor_SMD:CP_Elec_10x10.5 -> Capacitor_SMD:CP_Elec_6.3x7.7
- L601: value 22uH -> 220u; footprint Inductor_SMD:L_12x12mm_H8mm -> Inductor_SMD:L_Changjiang_FNR8065S
- L701: footprint Inductor_SMD:L_12x12mm_H8mm -> Inductor_SMD:L_Changjiang_FNR8065S; moved to B.Cu
- L801: footprint Inductor_SMD:L_12x12mm_H8mm -> Inductor_SMD:L_Changjiang_FNR8065S
- moved U701 137.5 mm to (73.2, 62.4)
- moved C702 134.6 mm to (64.0, 67.5)
- moved R701 131.3 mm to (66.0, 67.5), turned to 180 degrees
- moved R703 121.0 mm to (64.1, 56.1), turned to 180 degrees
- moved C501 120.7 mm to (79.8, 66.5)
- moved C502 120.7 mm to (85.1, 66.0)
- moved U501 120.7 mm to (82.5, 67.0)
- moved R501 120.7 mm to (85.0, 67.8)
- moved D501 117.6 mm to (86.4, 67.2), turned to -90 degrees
- moved R702 116.3 mm to (66.0, 56.1), turned to 180 degrees
- moved R109 112.5 mm to (87.7, 52.0), turned to -90 degrees
- moved R114 112.5 mm to (87.7, 54.0)
- moved CR701 111.9 mm to (74.1, 65.5), turned to 90 degrees
- moved D104 110.2 mm to (85.6, 52.5), turned to 180 degrees
- moved R106 107.7 mm to (87.7, 50.1), turned to -90 degrees
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Connections:
- IC101 pad 25: /FDC_6 -> /FDC_7
- IC101 pad 26: /FDC_7 -> /FDC_6
Routing:
- net GND1: track 180.7 -> 123.7 mm, vias 33 -> 32
- net /FDC_2: track 1.97 -> 31.5 mm, vias 0 -> 2
- net +3.3V: track 59.1 -> 85.8 mm, vias 1 -> 8
- net 7.5V: track 36.5 -> 9.94 mm
- net 24V: track 41.7 -> 65.9 mm, vias 33 -> 108
- net 5.1V: track 35.2 -> 55.3 mm, vias 1 -> 32
- net /Régulateur 11.7V/Vsw: track 0.00 -> 16.5 mm, vias 0 -> 2
- net Net-(J102-Pin_2): track 0.00 -> 15.6 mm
- net Net-(U701-FB): track 0.00 -> 13.1 mm, vias 0 -> 2
- net 11.7V: track 0.00 -> 9.59 mm, vias 0 -> 1
- net Net-(U701-Vc): track 0.00 -> 4.88 mm
- net /Régulateur 7.5V/Vsw: track 21.1 -> 16.5 mm, vias 1 -> 2
- net Net-(U801-FB): track 8.92 -> 13.4 mm, vias 0 -> 2
- net Net-(Q101-G): track 0.00 -> 4.38 mm
- net /Régulateur 5.1V/Vsw: track 18.8 -> 15.3 mm, vias 1 -> 2
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- added copper zone on B.Cu, net +3.3V
- added copper zone on In1.Cu, net +3.3V
- added copper zone on F.Cu, net 24V
- added copper zone on In1.Cu, net 24V
- added copper zone on In2.Cu, net 5.1V
- added copper zone on In2.Cu, net GND1
- removed copper zone on In1.Cu, net GND1

Commit message: updata cha 20/12
Parts:
- moved D501 1.17 mm to (87.5, 67.0)
- moved J109 1.15 mm to (92.6, 60.5)
- moved C501 0.58 mm to (80.3, 66.3)
- moved C502 0.58 mm to (85.6, 65.7)
- moved U501 0.58 mm to (83.0, 66.8)
- moved R501 0.58 mm to (85.6, 67.6)
- moved J110 0.45 mm to (25.8, 47.9)
- moved Q101 0.35 mm to (22.7, 42.7)
- moved D601 0.25 mm to (82.5, 52.8)
- moved R107 0.20 mm to (26.6, 42.4)
- moved R108 0.20 mm to (26.6, 41.4)
- moved J103 0.18 mm to (24.1, 37.0)
- moved R604 0.15 mm to (80.0, 52.7)
- moved R119 0.10 mm to (80.0, 47.7), turned to 0 degrees
- moved D701 0.10 mm to (82.5, 49.4)
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Routing:
- net 24V: track 65.9 -> 66.9 mm
- net Net-(D501-A): track 1.46 -> 2.47 mm
- net GND1: track 123.7 -> 123.9 mm, vias 32 -> 34
- net 5.1V: track 55.3 -> 55.5 mm, vias 32 -> 28
