File: Kicad/Eve/Reg2.kicad_sch (KiCad schematic)
At the start: 9 parts

Commit message: updtated Kicad ver 7.11.23
Parts:
- removed C32: 220uF, Capacitor_SMD:CP_Elec_10x10.5, symbol Device:C_Polarized_Small
- removed C33: 10n, Capacitor_SMD:C_0603_1608Metric_Pad1.08x0.95mm_HandSolder, symbol Device:C_Small
- removed C34: 470uF, Capacitor_SMD:CP_Elec_10x10.5, symbol Device:C_Polarized_Small
- removed CR2: DST10100S, libs:DST10100S, symbol 2023-03-19_11-33-54:DST10100S
- removed L3: 22uH, Inductor_SMD:L_Wuerth_WE-PD-Typ-LS_Handsoldering, symbol Device:L_Small
- removed R14: 2.7k, Resistor_SMD:R_0603_1608Metric_Pad0.98x0.95mm_HandSolder, symbol Device:R_Small
- removed U6: ~, libs:LT1076CR-PBF, symbol custom:LT1076
- added C6: 220uF, Capacitor_SMD:CP_Elec_10x10.5, symbol Device:C_Polarized_Small
- added C7: 10n, Capacitor_SMD:C_0603_1608Metric_Pad1.08x0.95mm_HandSolder, symbol Device:C_Small
- added C8: 470uF, Capacitor_SMD:CP_Elec_10x10.5, symbol Device:C_Polarized_Small
- added CR1: DST10100S, TO277B_LTF, symbol 2023-03-19_11-33-54:DST10100S
- added D5: LED, LED_SMD:LED_0603_1608Metric_Pad1.05x0.95mm_HandSolder, symbol Device:LED
- added L1: 22uH, Inductor_SMD:L_Wuerth_WE-PD-Typ-LS_Handsoldering, symbol Device:L_Small
- added R6: 1k, Resistor_SMD:R_0603_1608Metric_Pad0.98x0.95mm_HandSolder, symbol Device:R_Small
- added R8: 2.7k, Resistor_SMD:R_0603_1608Metric_Pad0.98x0.95mm_HandSolder, symbol Device:R_Small
- added U1: ~, symbol custom:LT1076
Connections:
- net +5.1V: now also C8.1, L1.2, R6.1
- net GND: now also C6.2, C7.2, C8.2, CR1.1, CR1.2, D5.1 (K), U1.4 (GND)
- net Vsw: now also CR1.3, L1.1, U1.2 (Vsw)
- net at R15.2, R16.1: now also U1.5 (FB)
- new net: D5.2 (A), R6.2
- new net: C7.1, R8.2
- new net: R8.1, U1.6 (Vc)
- new net 24V: C6.1, U1.1 (Vin), U1.7 (Shutdown)
Other:
- moved on the sheet: R16

Commit message: added Kicad libraries to git + sch changes 11/11/23
Changed lines of the file:
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@@
   (junction (at 146.05 69.85) (diameter 0) (color 0 0 0 0)
-  )
-  (junction (at 156.21 69.85) (diameter 0) (color 0 0 0 0)
   )
   (junction (at 143.51 95.25) (diameter 0) (color 0 0 0 0)
@@
   )
   (wire (pts (xy 105.41 81.28) (xy 105.41 85.09))
-    (stroke (width 0) (type default))
-  )
-  (wire (pts (xy 156.21 69.85) (xy 170.18 69.85))
     (stroke (width 0) (type default))
   )
@@
     (effects (font (size 1.27 1.27)) (justify left bottom))
   )
-  (label "5.1V" (at 205.74 74.93 0) (fields_autoplaced)
-    (effects (font (size 1.27 1.27)) (justify left bottom))
-  )
-  (label "Vin" (at 101.6 73.66 0) (fields_autoplaced)
-    (effects (font (size 1.27 1.27)) (justify left bottom))
-  )
-  (label "5.1V" (at 165.1 69.85 0) (fields_autoplaced)
-    (effects (font (size 1.27 1.27)) (justify left bottom))
-  )
   (label "Vsw" (at 135.89 72.39 180) (fields_autoplaced)
     (effects (font (size 1.27 1.27)) (justify right bottom))
-  )
-  (label "Vout" (at 158.75 69.85 0) (fields_autoplaced)
-    (effects (font (size 1.27 1.27)) (justify left bottom))
   )
   (hierarchical_label "24V" (shape input) (at 96.52 72.39 90) (fields_autoplaced)
     (effects (font (size 1.27 1.27)) (justify left))
   )
-  (hierarchical_label "+5.1V" (shape input) (at 170.18 69.85 0) (fields_autoplaced)
+  (hierarchical_label "+5.1V" (shape input) (at 156.21 69.85 0) (fields_autoplaced)
     (effects (font (size 1.27 1.27)) (justify left))
   )
+  (hierarchical_label "+5.1V" (shape input) (at 205.74 74.93 90) (fields_autoplaced)
+    (effects (font (size 1.27 1.27)) (justify left))
+  )

Commit message: empreinte 13/11
Parts:
- C6: value 220uF -> 220u; footprint Capacitor_SMD:CP_Elec_10x10.5 -> (none)
- C8: value 470uF -> 470u; footprint Capacitor_SMD:CP_Elec_10x10.5 -> (none)
- CR1: footprint TO277B_LTF -> libs:DST10100S
- L1: footprint Inductor_SMD:L_Wuerth_WE-PD-Typ-LS_Handsoldering -> (none)
- U1: footprint (none) -> libs:LT1076CR-PBF
Changed lines of the file:
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@@
       (effects (font (size 1.524 1.524)) (justify right))
     )
-    (property "Footprint" "TO277B_LTF" (at 132.334 82.55 0)
+    (property "Footprint" "libs:DST10100S" (at 132.334 82.55 0)
       (effects (font (size 1.524 1.524)) hide)
     )
@@
       (effects (font (size 1.27 1.27)) (justify left))
     )
-    (property "Value" "470uF" (at 148.59 80.01 0)
-      (effects (font (size 1.27 1.27)) (justify left))
-    )
-    (property "Footprint" "Capacitor_SMD:CP_Elec_10x10.5" (at 146.05 78.74 0)
+    (property "Value" "470u" (at 148.59 80.01 0)
+      (effects (font (size 1.27 1.27)) (justify left))
+    )
+    (property "Footprint" "" (at 146.05 78.74 0)
       (effects (font (size 1.27 1.27)) hide)
     )
@@
       (effects (font (size 1.27 1.27)) (justify left))
     )
-    (property "Value" "220uF" (at 97.79 82.4611 0)
-      (effects (font (size 1.27 1.27)) (justify left))
-    )
-    (property "Footprint" "Capacitor_SMD:CP_Elec_10x10.5" (at 105.41 78.74 0)
+    (property "Value" "220u" (at 97.79 82.4611 0)
+      (effects (font (size 1.27 1.27)) (justify left))
+    )
+    (property "Footprint" "" (at 105.41 78.74 0)
       (effects (font (size 1.27 1.27)) hide)
     )
@@
       (effects (font (size 1.27 1.27)))
     )
-    (property "Footprint" "" (at 116.84 77.47 0)
+    (property "Footprint" "libs:LT1076CR-PBF" (at 116.84 77.47 0)
       (effects (font (size 1.27 1.27)) hide)
     )
@@
       (effects (font (size 1.27 1.27)))
     )
-    (property "Footprint" "Inductor_SMD:L_Wuerth_WE-PD-Typ-LS_Handsoldering" (at 142.24 69.85 0)
-      (effects (font (size 1.27 1.27)) hide)
-    )
+    (property "Footprint" "" (at 142.24 69.85 0)
+      (effects (font (size 1.27 1.27)) hide)
+    )

Commit message: pulled main and started routing
Parts:
- C6, C8: footprint (none) -> Capacitor_SMD:CP_Elec_10x10.5
- L1: footprint (none) -> Eagle_WE-PD (rev23a):WE-PD_1210
Changed lines of the file:
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@@
       (effects (font (size 1.27 1.27)) (justify left))
     )
-    (property "Footprint" "" (at 146.05 78.74 0)
+    (property "Footprint" "Capacitor_SMD:CP_Elec_10x10.5" (at 146.05 78.74 0)
       (effects (font (size 1.27 1.27)) hide)
     )
@@
       (effects (font (size 1.27 1.27)) (justify left))
     )
-    (property "Footprint" "" (at 105.41 78.74 0)
+    (property "Footprint" "Capacitor_SMD:CP_Elec_10x10.5" (at 105.41 78.74 0)
       (effects (font (size 1.27 1.27)) hide)
     )
@@
       (effects (font (size 1.27 1.27)))
     )
-    (property "Footprint" "" (at 142.24 69.85 0)
-      (effects (font (size 1.27 1.27)) hide)
-    )
+    (property "Footprint" "Eagle_WE-PD (rev23a):WE-PD_1210" (at 142.24 69.85 0)
+      (effects (font (size 1.27 1.27)) hide)
+    )

Commit message: update pcb
Parts:
- C?: renamed from C7; footprint Capacitor_SMD:C_0603_1608Metric_Pad1.08x0.95mm_HandSolder -> Capacitor_SMD:C_0402_1005Metric
- CR?: renamed from CR1; footprint libs:DST10100S -> DST10100S:DST10100S
- D?: renamed from D5; footprint LED_SMD:LED_0603_1608Metric_Pad1.05x0.95mm_HandSolder -> LED_SMD:LED_0603_1608Metric
- L?: renamed from L1; footprint Eagle_WE-PD (rev23a):WE-PD_1210 -> Inductor_SMD:L_12x12mm_H8mm
- R602: renamed from R15; footprint Resistor_SMD:R_0603_1608Metric_Pad0.98x0.95mm_HandSolder -> Resistor_SMD:R_0402_1005Metric
- R603: renamed from R16; footprint Resistor_SMD:R_0603_1608Metric_Pad0.98x0.95mm_HandSolder -> Resistor_SMD:R_0402_1005Metric
- R?: renamed from R6; footprint Resistor_SMD:R_0603_1608Metric_Pad0.98x0.95mm_HandSolder -> Resistor_SMD:R_0402_1005Metric
- R?: renamed from R8; footprint Resistor_SMD:R_0603_1608Metric_Pad0.98x0.95mm_HandSolder -> Resistor_SMD:R_0402_1005Metric
- U?: renamed from U1; value ~ -> LT1076CR-PBF; footprint libs:LT1076CR-PBF -> LT1076CR:LT1076CR-PBF
- renumbered C8 to C?, C6 to C?

Commit message: update PCB
Parts:
- removed C?: 220u, Capacitor_SMD:CP_Elec_10x10.5, symbol Device:C_Polarized_Small
- added C?: 100u, Capacitor_SMD:CP_Elec_6.3x7.7, symbol Device:C_Polarized_Small
- C?: value 470u -> 47u; footprint Capacitor_SMD:CP_Elec_10x10.5 -> Capacitor_SMD:CP_Elec_6.3x5.4; MFR 865060457009 -> 865060543005
- L?: value 22uH -> 220u; footprint Inductor_SMD:L_12x12mm_H8mm -> Inductor_SMD:L_Changjiang_FNR8065S; MFR 7447709220 -> 74404086221
Connections:
- net 24V: now also C?.1
- net GND: now also C?.2
Changed lines of the file:
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@@
+    )
+  )
+  (symbol (lib_id "Device:C_Polarized_Small") (at 105.41 78.74 0) (unit 1)
+    (in_bom yes) (on_board yes) (dnp no)
+    (property "Reference" "C?" (at 100.33 80.01 0)
+      (effects (font (size 1.27 1.27)) (justify left))
+    )
+    (property "Value" "100u" (at 97.79 82.4611 0)
+      (effects (font (size 1.27 1.27)) (justify left))
+    )
+    (property "Footprint" "Capacitor_SMD:CP_Elec_6.3x7.7" (at 105.41 78.74 0)
+      (effects (font (size 1.27 1.27)) hide)
+    )
+    (property "Datasheet" "~" (at 105.41 78.74 0)
+      (effects (font (size 1.27 1.27)) hide)
+    )
+    (property "MFR" "865060445005" (at 105.41 78.74 0)
+      (effects (font (size 1.27 1.27)) hide)
+    )
+    (property "Vmax" "25V" (at 105.41 78.74 0)
+      (effects (font (size 1.27 1.27)) hide)
+    )
+    (pin "1")
+    (pin "2")
+    (instances
+      (project "Robourt"
+        (path "/87ede840-4957-4951-b25a-c132e7988ddc/45a40ff7-b6ec-4165-9635-bd80258dd043"
+          (reference "C?") (unit 1)
+        )
+        (path "/87ede840-4957-4951-b25a-c132e7988ddc/b0f3c6bf-43ee-43a7-9a34-92e1e933f121"
+          (reference "C801") (unit 1)
+        )
+        (path "/87ede840-4957-4951-b25a-c132e7988ddc/c08e9c7d-1604-43bb-a00c-546e3bb44d34"
+          (reference "C704") (unit 1)
+        )
+        (path "/87ede840-4957-4951-b25a-c132e7988ddc/9b84e365-6524-43b0-9106-e6e67f034906"
+          (reference "C604") (unit 1)
+        )
+      )
+      (project "Regulateurs"
+        (path "/c482be3d-70a8-4e95-a602-5f49202f2a67"
+          (reference "C?") (unit 1)
+        )
+      )
+      (project "QBPS_LT1076CR#PBF"
+        (path "/d1da92a7-0236-4679-a8f0-7224ece43232/caa3dddc-44de-4526-a352-aeb906051043"
+          (reference "C?") (unit 1)
+        )
+        (path "/d1da92a7-0236-4679-a8f0-7224ece43232/13fecffc-9de7-4a7f-bbf5-bc48726faeaa"
+          (reference "C?") (unit 1)
+        )
+        (path "/d1da92a7-0236-4679-a8f0-7224ece43232/62fde565-aeb8-4b1e-8686-1a60119375b4"
+          (reference "C?") (unit 1)
+        )
+        (path "/d1da92a7-0236-4679-a8f0-7224ece43232/19a5ec18-751a-4622-82f3-c22b8bd4516c"
+          (reference "C?") (unit 1)
+        )
+      )
     )
   )
@@
       (effects (font (size 1.27 1.27)) (justify left))
     )
-    (property "Value" "470u" (at 148.59 80.01 0)
-      (effects (font (size 1.27 1.27)) (justify left))
-    )
-    (property "Footprint" "Capacitor_SMD:CP_Elec_10x10.5" (at 146.05 78.74 0)
+    (property "Value" "47u" (at 148.59 80.01 0)
+      (effects (font (size 1.27 1.27)) (justify left))
+    )
+    (property "Footprint" "Capacitor_SMD:CP_Elec_6.3x5.4" (at 146.05 78.74 0)
       (effects (font (size 1.27 1.27)) hide)
     )
@@
       (effects (font (size 1.27 1.27)) hide)
     )
-    (property "MFR" "865060457009" (at 146.05 78.74 0)
+    (property "MFR" "865060543005" (at 146.05 78.74 0)
       (effects (font (size 1.27 1.27)) hide)
     )
@@
         (path "/d1da92a7-0236-4679-a8f0-7224ece43232/19a5ec18-751a-4622-82f3-c22b8bd4516c"
           (reference "R?") (unit 1)
-        )
-      )
-    )
-  )
-  (symbol (lib_id "Device:C_Polarized_Small") (at 105.41 78.74 0) (unit 1)
-    (in_bom yes) (on_board yes) (dnp no)
-    (property "Reference" "C?" (at 100.33 80.01 0)
-      (effects (font (size 1.27 1.27)) (justify left))
-    )
-    (property "Value" "220u" (at 97.79 82.4611 0)
-      (effects (font (size 1.27 1.27)) (justify left))
-    )
-    (property "Footprint" "Capacitor_SMD:CP_Elec_10x10.5" (at 105.41 78.74 0)
-      (effects (font (size 1.27 1.27)) hide)
-    )
-    (property "Datasheet" "~" (at 105.41 78.74 0)
-      (effects (font (size 1.27 1.27)) hide)
-    )
-    (property "MFR" "865060657012" (at 105.41 78.74 0)
-      (effects (font (size 1.27 1.27)) hide)
-    )
-    (property "Vmax" "50V" (at 105.41 78.74 0)
-      (effects (font (size 1.27 1.27)) hide)
-    )
-    (pin "1")
-    (pin "2")
-    (instances
-      (project "Robourt"
-        (path "/87ede840-4957-4951-b25a-c132e7988ddc/45a40ff7-b6ec-4165-9635-bd80258dd043"
-          (reference "C?") (unit 1)
-        )
-        (path "/87ede840-4957-4951-b25a-c132e7988ddc/9b84e365-6524-43b0-9106-e6e67f034906"
-          (reference "C601") (unit 1)
-        )
-      )
-      (project "Regulateurs"
-        (path "/c482be3d-70a8-4e95-a602-5f49202f2a67"
-          (reference "C?") (unit 1)
-        )
-      )
-      (project "QBPS_LT1076CR#PBF"
-        (path "/d1da92a7-0236-4679-a8f0-7224ece43232/caa3dddc-44de-4526-a352-aeb906051043"
-          (reference "C?") (unit 1)
-        )
-        (path "/d1da92a7-0236-4679-a8f0-7224ece43232/13fecffc-9de7-4a7f-bbf5-bc48726faeaa"
-          (reference "C?") (unit 1)
-        )
-        (path "/d1da92a7-0236-4679-a8f0-7224ece43232/62fde565-aeb8-4b1e-8686-1a60119375b4"
-          (reference "C?") (unit 1)
-        )
-        (path "/d1da92a7-0236-4679-a8f0-7224ece43232/19a5ec18-751a-4622-82f3-c22b8bd4516c"
-          (reference "C?") (unit 1)
         )
       )
@@
       (effects (font (size 1.27 1.27)))
     )
-    (property "Value" "22uH" (at 142.24 68.58 90)
-      (effects (font (size 1.27 1.27)))
-    )
-    (property "Footprint" "Inductor_SMD:L_12x12mm_H8mm" (at 142.24 69.85 0)
+    (property "Value" "220u" (at 142.24 68.58 90)
+      (effects (font (size 1.27 1.27)))
+    )
+    (property "Footprint" "Inductor_SMD:L_Changjiang_FNR8065S" (at 142.24 69.85 0)
       (effects (font (size 1.27 1.27)) hide)
     )
@@
       (effects (font (size 1.27 1.27)) hide)
     )
-    (property "MFR" "7447709220" (at 142.24 69.85 90)
-      (effects (font (size 1.27 1.27)) hide)
-    )
+    (property "MFR" "74404086221" (at 142.24 69.85 90)
+      (effects (font (size 1.27 1.27)) hide)
+    )
