File: Kicad/Eve/reg3.kicad_sch (KiCad schematic)
At the start: 11 parts

Commit message: update pcb
Parts:
- C?: renamed from C7; footprint Capacitor_SMD:C_0603_1608Metric_Pad1.08x0.95mm_HandSolder -> Capacitor_SMD:C_0402_1005Metric
- CR?: renamed from CR1; footprint libs:DST10100S -> DST10100S:DST10100S
- D?: renamed from D3; footprint LED_SMD:LED_0603_1608Metric_Pad1.05x0.95mm_HandSolder -> LED_SMD:LED_0603_1608Metric
- L?: renamed from L1; footprint Eagle_WE-PD (rev23a):WE-PD_1210 -> Inductor_SMD:L_12x12mm_H8mm
- R702: renamed from R12; footprint Resistor_SMD:R_0603_1608Metric_Pad0.98x0.95mm_HandSolder -> Resistor_SMD:R_0402_1005Metric
- R703: renamed from R13; footprint Resistor_SMD:R_0603_1608Metric_Pad0.98x0.95mm_HandSolder -> Resistor_SMD:R_0402_1005Metric
- R?: renamed from R4; footprint Resistor_SMD:R_0603_1608Metric_Pad0.98x0.95mm_HandSolder -> Resistor_SMD:R_0402_1005Metric
- R?: renamed from R8; footprint Resistor_SMD:R_0603_1608Metric_Pad0.98x0.95mm_HandSolder -> Resistor_SMD:R_0402_1005Metric
- U?: renamed from U1; value ~ -> LT1076CR-PBF; footprint libs:LT1076CR-PBF -> LT1076CR:LT1076CR-PBF
- renumbered C6 to C?, C8 to C?

Commit message: update 18/12
Parts:
- R?: value 680 -> 2k
Changed lines of the file:
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@@
   (symbol (lib_id "Device:R_Small") (at 229.87 85.09 0) (unit 1)
     (in_bom yes) (on_board yes) (dnp no) (fields_autoplaced)
-    (property "Reference" "R?" (at 232.41 83.82 0)
+    (property "Reference" "R?" (at 232.41 84.455 0)
       (effects (font (size 1.27 1.27)) (justify left))
     )
-    (property "Value" "680" (at 232.41 86.36 0)
+    (property "Value" "2k" (at 232.41 86.995 0)
       (effects (font (size 1.27 1.27)) (justify left))
     )

Commit message: update PCB
Parts:
- removed C?: 220u, Capacitor_SMD:CP_Elec_10x10.5, symbol Device:C_Polarized_Small
- added C?: 100u, Capacitor_SMD:CP_Elec_6.3x7.7, symbol Device:C_Polarized_Small
- C?: value 470u -> 47u; footprint Capacitor_SMD:CP_Elec_10x10.5 -> Capacitor_SMD:CP_Elec_6.3x5.4; MFR 865060457009 -> 865060543005
- L?: footprint Inductor_SMD:L_12x12mm_H8mm -> Inductor_SMD:L_Changjiang_FNR8065S
Connections:
- net 24V: now also C?.1
- net GND: now also C?.2
Changed lines of the file:
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@@
       (effects (font (size 1.27 1.27)))
     )
-    (property "Footprint" "Inductor_SMD:L_12x12mm_H8mm" (at 142.24 76.2 0)
+    (property "Footprint" "Inductor_SMD:L_Changjiang_FNR8065S" (at 142.24 76.2 0)
       (effects (font (size 1.27 1.27)) hide)
     )
@@
     )
   )
+  (symbol (lib_id "Device:C_Polarized_Small") (at 105.41 85.09 0) (unit 1)
+    (in_bom yes) (on_board yes) (dnp no)
+    (property "Reference" "C?" (at 100.33 86.36 0)
+      (effects (font (size 1.27 1.27)) (justify left))
+    )
+    (property "Value" "100u" (at 97.79 88.8111 0)
+      (effects (font (size 1.27 1.27)) (justify left))
+    )
+    (property "Footprint" "Capacitor_SMD:CP_Elec_6.3x7.7" (at 105.41 85.09 0)
+      (effects (font (size 1.27 1.27)) hide)
+    )
+    (property "Datasheet" "~" (at 105.41 85.09 0)
+      (effects (font (size 1.27 1.27)) hide)
+    )
+    (property "MFR" "865060445005" (at 105.41 85.09 0)
+      (effects (font (size 1.27 1.27)) hide)
+    )
+    (property "Vmax" "25V" (at 105.41 85.09 0)
+      (effects (font (size 1.27 1.27)) hide)
+    )
+    (pin "1")
+    (pin "2")
+    (instances
+      (project "Robourt"
+        (path "/87ede840-4957-4951-b25a-c132e7988ddc/45a40ff7-b6ec-4165-9635-bd80258dd043"
+          (reference "C?") (unit 1)
+        )
+        (path "/87ede840-4957-4951-b25a-c132e7988ddc/b0f3c6bf-43ee-43a7-9a34-92e1e933f121"
+          (reference "C801") (unit 1)
+        )
+        (path "/87ede840-4957-4951-b25a-c132e7988ddc/c08e9c7d-1604-43bb-a00c-546e3bb44d34"
+          (reference "C704") (unit 1)
+        )
+      )
+      (project "Regulateurs"
+        (path "/c482be3d-70a8-4e95-a602-5f49202f2a67"
+          (reference "C?") (unit 1)
+        )
+      )
+      (project "QBPS_LT1076CR#PBF"
+        (path "/d1da92a7-0236-4679-a8f0-7224ece43232/caa3dddc-44de-4526-a352-aeb906051043"
+          (reference "C?") (unit 1)
+        )
+        (path "/d1da92a7-0236-4679-a8f0-7224ece43232/13fecffc-9de7-4a7f-bbf5-bc48726faeaa"
+          (reference "C?") (unit 1)
+        )
+        (path "/d1da92a7-0236-4679-a8f0-7224ece43232/62fde565-aeb8-4b1e-8686-1a60119375b4"
+          (reference "C?") (unit 1)
+        )
+        (path "/d1da92a7-0236-4679-a8f0-7224ece43232/19a5ec18-751a-4622-82f3-c22b8bd4516c"
+          (reference "C?") (unit 1)
+        )
+      )
+    )
+  )
   (symbol (lib_id "power:GND") (at 143.51 101.6 0) (unit 1)
     (in_bom yes) (on_board yes) (dnp no)
@@
     )
   )
-  (symbol (lib_id "Device:C_Polarized_Small") (at 105.41 85.09 0) (unit 1)
-    (in_bom yes) (on_board yes) (dnp no)
-    (property "Reference" "C?" (at 100.33 86.36 0)
-      (effects (font (size 1.27 1.27)) (justify left))
-    )
-    (property "Value" "220u" (at 97.79 88.8111 0)
-      (effects (font (size 1.27 1.27)) (justify left))
-    )
-    (property "Footprint" "Capacitor_SMD:CP_Elec_10x10.5" (at 105.41 85.09 0)
-      (effects (font (size 1.27 1.27)) hide)
-    )
-    (property "Datasheet" "~" (at 105.41 85.09 0)
-      (effects (font (size 1.27 1.27)) hide)
-    )
-    (property "MFR" "865060657012" (at 105.41 85.09 0)
-      (effects (font (size 1.27 1.27)) hide)
-    )
-    (property "Vmax" "50V" (at 105.41 85.09 0)
-      (effects (font (size 1.27 1.27)) hide)
-    )
-    (pin "1")
-    (pin "2")
-    (instances
-      (project "Robourt"
-        (path "/87ede840-4957-4951-b25a-c132e7988ddc/45a40ff7-b6ec-4165-9635-bd80258dd043"
-          (reference "C?") (unit 1)
-        )
-        (path "/87ede840-4957-4951-b25a-c132e7988ddc/c08e9c7d-1604-43bb-a00c-546e3bb44d34"
-          (reference "C701") (unit 1)
-        )
-      )
-      (project "Regulateurs"
-        (path "/c482be3d-70a8-4e95-a602-5f49202f2a67"
-          (reference "C?") (unit 1)
-        )
-      )
-      (project "QBPS_LT1076CR#PBF"
-        (path "/d1da92a7-0236-4679-a8f0-7224ece43232/caa3dddc-44de-4526-a352-aeb906051043"
-          (reference "C?") (unit 1)
-        )
-        (path "/d1da92a7-0236-4679-a8f0-7224ece43232/13fecffc-9de7-4a7f-bbf5-bc48726faeaa"
-          (reference "C?") (unit 1)
-        )
-        (path "/d1da92a7-0236-4679-a8f0-7224ece43232/62fde565-aeb8-4b1e-8686-1a60119375b4"
-          (reference "C?") (unit 1)
-        )
-        (path "/d1da92a7-0236-4679-a8f0-7224ece43232/19a5ec18-751a-4622-82f3-c22b8bd4516c"
-          (reference "C?") (unit 1)
-        )
-      )
-    )
-  )
   (symbol (lib_id "Device:C_Polarized_Small") (at 146.05 85.09 0) (unit 1)
     (in_bom yes) (on_board yes) (dnp no)
@@
       (effects (font (size 1.27 1.27)) (justify left))
     )
-    (property "Value" "470u" (at 148.59 86.36 0)
-      (effects (font (size 1.27 1.27)) (justify left))
-    )
-    (property "Footprint" "Capacitor_SMD:CP_Elec_10x10.5" (at 146.05 85.09 0)
+    (property "Value" "47u" (at 148.59 86.36 0)
+      (effects (font (size 1.27 1.27)) (justify left))
+    )
+    (property "Footprint" "Capacitor_SMD:CP_Elec_6.3x5.4" (at 146.05 85.09 0)
       (effects (font (size 1.27 1.27)) hide)
     )
@@
       (effects (font (size 1.27 1.27)) hide)
     )
-    (property "MFR" "865060457009" (at 146.05 85.09 0)
-      (effects (font (size 1.27 1.27)) hide)
-    )
+    (property "MFR" "865060543005" (at 146.05 85.09 0)
+      (effects (font (size 1.27 1.27)) hide)
+    )
